Commit message: Fix names

File: xacro/leg.xacro (robot description, xacro)
@@ -21,5 +21,5 @@
     <joint name="${prefix}_hfe_joint" type="revolute">
       <parent link="trunk"/>
-      <child link="${prefix}_UPPER_LEG"/>
+      <child link="${prefix}_upper_leg"/>
       <limit effort="1000" lower="-10" upper="10" velocity="1000"/>
       <!-- joints rotates around the y-axis -->
@@ -46,5 +46,5 @@
     </joint>
     <!-- UPPER LEG LINK -->
-    <link name="${prefix}_UPPER_LEG">
+    <link name="${prefix}_upper_leg">
       <!-- UPPER LEG LINK INERTIAL -->
       <xacro:unless value="${is_right}">
@@ -106,6 +106,6 @@
     <!-- KFE JOINT -->
     <joint name="${prefix}_kfe_joint" type="revolute">
-      <parent link="${prefix}_UPPER_LEG"/>
-      <child link="${prefix}_LOWER_LEG"/>
+      <parent link="${prefix}_upper_leg"/>
+      <child link="${prefix}_lower_leg"/>
       <limit effort="1000" lower="-10" upper="10" velocity="1000"/>
       <!-- joints rotates around the y-axis -->
@@ -132,5 +132,5 @@
     </joint>
     <!-- LOWERLEG -->
-    <link name="${prefix}_LOWER_LEG">
+    <link name="${prefix}_lower_leg">
       <!-- LOWER LEG LINK INERTIAL -->
       <xacro:unless value="${is_right}">
@@ -191,7 +191,7 @@
     </link> <!-- END LOWER LEG LINK -->
 <!-- KFE: Joint between the upper leg and the lower leg -->
-<joint name="${prefix}_ANKLE" type="fixed">
-  <parent link="${prefix}_LOWER_LEG"/>
-  <child link="${prefix}_FOOT"/>
+<joint name="${prefix}_ankle" type="fixed">
+  <parent link="${prefix}_lower_leg"/>
+  <child link="${prefix}_foot"/>
   <!-- Joint placement -->
   <origin xyz="0 0 ${-HFE_2_KFE_z}" rpy="0 0 0" />
