Commit message: corrected some stuff

File: urdfs/leg.gazebo.xacro (robot description, xacro)
@@ -2,17 +2,4 @@
 <robot xmlns:xacro="http://ros.org/wiki/xacro">
         <xacro:macro name="leg_gazebo" params="name load_force_sensors">
-                <gazebo reference="${name}_haa_joint">
-                        <provideFeedback>true</provideFeedback>
-                </gazebo>
-                <xacro:if value="${load_force_sensors}">
-                        <gazebo>
-                                <plugin name="${name}_haa_sensor" filename="libgazebo_ros_ft_sensor.so">
-                                        <robotNamespace>/hyq/internal_wrench/</robotNamespace>
-                                        <updateRate>100.0</updateRate>
-                                        <topicName>${name}_haa_joint</topicName>
-                                        <jointName>${name}_haa_joint</jointName>
-                                </plugin>
-                        </gazebo>
-                </xacro:if>
                 <gazebo reference="${name}_kfe_joint">
                         <provideFeedback>true</provideFeedback>
@@ -21,5 +8,5 @@
                         <gazebo>
                                 <plugin name="${name}_kfe_sensor" filename="libgazebo_ros_ft_sensor.so">
-                                        <robotNamespace>/hyq/internal_wrench/</robotNamespace>
+                                        <robotNamespace>/solo/internal_wrench/</robotNamespace>
                                         <updateRate>100.0</updateRate>
                                         <topicName>${name}_kfe_joint</topicName>
@@ -34,5 +21,5 @@
                         <gazebo>
                                 <plugin name="${name}_hfe_sensor" filename="libgazebo_ros_ft_sensor.so">
-                                        <robotNamespace>/hyq/internal_wrench/</robotNamespace>
+                                        <robotNamespace>/solo/internal_wrench/</robotNamespace>
                                         <updateRate>100.0</updateRate>
                                         <topicName>${name}_hfe_joint</topicName>
@@ -66,5 +53,5 @@
                 because gazebo lumps the fake footframe with the real parent link, the normals are in the world frame-->
                  <plugin name="${name}_shin_bumper" filename="libgazebo_ros_bumper.so">
-                  <bumperTopicName>/hyq/${name}_shin_bumper</bumperTopicName>
+                  <bumperTopicName>/solo/${name}_shin_bumper</bumperTopicName>
                 </plugin>
             </sensor>
@@ -86,6 +73,6 @@
                                 because gazebo lumps the fake footframe with the real parent link, the normals are in the world frame-->
                                 <plugin name="${name}_foot_bumper" filename="libgazebo_ros_bumper.so">
-                                        <bumperTopicName>/hyq/${name}_foot_bumper</bumperTopicName>
-                                        <robotNamespace>hyq</robotNamespace>
+                                        <bumperTopicName>/solo/${name}_foot_bumper</bumperTopicName>
+                                        <robotNamespace>solo</robotNamespace>
                                 </plugin>
                         </sensor>

File: urdfs/leg.transmission.xacro (robot description, xacro)
@@ -2,15 +2,4 @@
 <robot xmlns:xacro="http://ros.org/wiki/xacro">
         <xacro:macro name="leg_transmission" params="name">
-        <!-- Hip assembly -->
-                <transmission name="${name}_haa_trans">
-                        <type>transmission_interface/SimpleTransmission</type>
-                        <joint name="${name}_haa_joint">
-                                <hardwareInterface>EffortJointInterface</hardwareInterface>
-                        </joint>
-                        <actuator name="${name}_haa_motor">
-                                <hardwareInterface>EffortJointInterface</hardwareInterface>
-                                <mechanicalReduction>1</mechanicalReduction>
-                        </actuator>
-                </transmission>
         <!-- Upper leg -->
                 <transmission name="${name}_hfe_trans">

File: xacro/leg.xacro (robot description, xacro)
@@ -2,6 +2,6 @@
 <robot xmlns:xacro="http://playerstage.sourceforge.net/gazebo/xmlschema/#interface" name="solo">
 <!-- Things that are needed only for Gazebo (not the physical robot). These include sensor and controller plugin specifications -->
-<!--<xacro:include filename="$(find solo_description)/urdfs/leg.transmission.xacro"/>
-<xacro:include filename="$(find solo_description)/urdfs/leg.gazebo.xacro"/>-->
+<xacro:include filename="$(find solo_description)/urdfs/leg.transmission.xacro"/>
+<xacro:include filename="$(find solo_description)/urdfs/leg.gazebo.xacro"/>
   <!-- See TODO: add the wiki link here -->
   <!-- These are absoulte distance value, the sign are decided below -->
@@ -239,6 +239,6 @@
     </link> <!-- END LOWER LEG LINK -->
         <!-- Extensions -->
-<!--        <xacro:leg_transmission name="${prefix}"/>
-        <xacro:leg_gazebo name="${prefix}" load_force_sensors="${load_force_sensors}"/>-->
+        <xacro:leg_transmission name="${prefix}"/>
+        <xacro:leg_gazebo name="${prefix}" load_force_sensors="${load_force_sensors}"/>
   </xacro:macro>
 </robot>

File: xacro/solo.urdf.xacro (robot description, xacro)
@@ -16,6 +16,6 @@
     </xacro:include>
     <!-- legs transmission -->
-<!--    <xacro:include filename="$(find solo_description)/urdfs/leg.transmission.xacro"/>
-    <xacro:include filename="$(find solo_description)/urdfs/leg.gazebo.xacro"/>-->
+    <xacro:include filename="$(find solo_description)/urdfs/leg.transmission.xacro"/>
+    <xacro:include filename="$(find solo_description)/urdfs/leg.gazebo.xacro"/>
     <!-- Material for the visual primitives -->
     <material name="solo_material">

Commit message: solo now has 12 dofs!

File: urdfs/leg.gazebo.xacro (robot description, xacro)
@@ -2,4 +2,17 @@
 <robot xmlns:xacro="http://ros.org/wiki/xacro">
         <xacro:macro name="leg_gazebo" params="name load_force_sensors">
+                <gazebo reference="${name}_haa_joint">
+                        <provideFeedback>true</provideFeedback>
+                </gazebo>
+                <xacro:if value="${load_force_sensors}">
+                        <gazebo>
+                                <plugin name="${name}_haa_sensor" filename="libgazebo_ros_ft_sensor.so">
+                                        <robotNamespace>/solo/internal_wrench/</robotNamespace>
+                                        <updateRate>100.0</updateRate>
+                                        <topicName>${name}_haa_joint</topicName>
+                                        <jointName>${name}_haa_joint</jointName>
+                                </plugin>
+                        </gazebo>
+                </xacro:if>
                 <gazebo reference="${name}_kfe_joint">
                         <provideFeedback>true</provideFeedback>

File: urdfs/leg.transmission.xacro (robot description, xacro)
@@ -2,4 +2,15 @@
 <robot xmlns:xacro="http://ros.org/wiki/xacro">
         <xacro:macro name="leg_transmission" params="name">
+        <!-- Hip assembly -->
+                <transmission name="${name}_haa_trans">
+                        <type>transmission_interface/SimpleTransmission</type>
+                        <joint name="${name}_haa_joint">
+                                <hardwareInterface>EffortJointInterface</hardwareInterface>
+                        </joint>
+                        <actuator name="${name}_haa_motor">
+                                <hardwareInterface>EffortJointInterface</hardwareInterface>
+                                <mechanicalReduction>1</mechanicalReduction>
+                        </actuator>
+                </transmission>
         <!-- Upper leg -->
                 <transmission name="${name}_hfe_trans">

File: xacro/leg.xacro (robot description, xacro)
@@ -10,39 +10,88 @@
   <xacro:property name="HFE_2_KFE_y" value="${37.45 * 0.001}" />
   <xacro:property name="HFE_2_KFE_z" value="${160.00 * 0.001}" />
-  <!-- To check this data to get the center of the foot properly -->
-  <xacro:property name="KFE_2_FOOT_y" value="${0.5 * 27.00 * 0.001}" />
+  <xacro:property name="KFE_2_FOOT_y" value="${8.0 * 0.001}" />
   <xacro:property name="KFE_2_FOOT_z" value="${160.00 * 0.001}" />
-  <xacro:property name="KFE_2_contact_y" value="${0 * 0.001}" />
-  <xacro:property name="KFE_2_contact_z" value="${(160.00 + 0.5*27) * 0.001}" />
   <!-- This macro has for purpose to define a left leg -->
-  <xacro:macro name="leg" params="prefix is_front is_right
+  <xacro:macro name="leg" params="prefix is_front is_right has_side_motion
                                   color_name color opacity load_force_sensors">
-    <!-- HFE JOINT -->
-    <joint name="${prefix}_hfe_joint" type="revolute">
-      <parent link="trunk"/>
-      <child link="${prefix}_upper_leg"/>
-      <limit effort="1000" lower="-10" upper="10" velocity="1000"/>
-      <!-- joints rotates around the y-axis -->
-      <axis xyz="0 1 0"/>
-      <!-- placement of the joint -->
-      <xacro:if value="${is_front}">
-        <xacro:unless value="${is_right}">
-          <origin xyz="${base_2_HFE_x} ${base_2_HFE_y} 0" rpy="0 0 0" />
-        </xacro:unless>
-        <xacro:if value="${is_right}">
-          <origin xyz="${base_2_HFE_x} ${-base_2_HFE_y} 0" rpy="0 0 0" />
-        </xacro:if>
-      </xacro:if>
-      <xacro:unless value="${is_front}">
-        <xacro:unless value="${is_right}">
-          <origin xyz="${-base_2_HFE_x} ${base_2_HFE_y} 0" rpy="0 0 0" />
-        </xacro:unless>
-        <xacro:if value="${is_right}">
-          <origin xyz="${-base_2_HFE_x} ${-base_2_HFE_y} 0" rpy="0 0 0" />
-        </xacro:if>
-      </xacro:unless>
-      <!-- pybullet simulation parameters -->
-      <dynamics damping="0.0" friction="0.0"/>
-    </joint>
+    <xacro:if value="${has_side_motion}">
+      <joint name="${prefix}_haa_joint" type="revolute">
+        <parent link="trunk"/>
+        <child link="${prefix}_hip_assembly"/>
+        <limit effort="1000" lower="-10" upper="10" velocity="1000"/>
+        <!-- joints rotates around the x-axis -->
+        <axis xyz="1 0 0"/>
+        <!-- placement of the joint -->
+        <xacro:if value="${is_front}">
+          <xacro:unless value="${is_right}">
+            <origin xyz="${base_2_HFE_x} ${base_2_HFE_y} 0" rpy="0 0 0" />
+          </xacro:unless>
+          <xacro:if value="${is_right}">
+            <origin xyz="${base_2_HFE_x} ${-base_2_HFE_y} 0" rpy="0 0 0" />
+          </xacro:if>
+        </xacro:if>
+        <xacro:unless value="${is_front}">
+          <xacro:unless value="${is_right}">
+            <origin xyz="${-base_2_HFE_x} ${base_2_HFE_y} 0" rpy="0 0 0" />
+          </xacro:unless>
+          <xacro:if value="${is_right}">
+            <origin xyz="${-base_2_HFE_x} ${-base_2_HFE_y} 0" rpy="0 0 0" />
+          </xacro:if>
+        </xacro:unless>
+        <!-- pybullet simulation parameters -->
+        <dynamics damping="0.0" friction="0.0"/>
+      </joint>
+      <link name="${prefix}_hip_assembly">
+        <!-- create a dummy hip_assembly link to join the two joints -->
+        <inertial>
+          <origin xyz="0. 0. 0." rpy="0 0 0" />
+          <!-- Adding extra weight for actuator module at hip_assembly. -->
+          <mass value="0.150"/>
+          <inertia ixx="0.00000001" ixy="0.0"        ixz="0.0"
+                                    iyy="0.00000001" iyz="0"
+                                                     izz="0.00000001"/>
+          </inertial>
+      </link>
+      <joint name="${prefix}_hfe_joint" type="revolute">
+        <parent link="${prefix}_hip_assembly"/>
+        <child link="${prefix}_upper_leg"/>
+        <limit effort="1000" lower="-10" upper="10" velocity="1000"/>
+        <!-- joints rotates around the y-axis -->
+        <axis xyz="0 1 0"/>
+        <!-- placement of the joint -->
+        <origin xyz="0 0 0" rpy="0 0 0" />
+        <!-- pybullet simulation parameters -->
+        <dynamics damping="0.0" friction="0.0"/>
+      </joint>
+    </xacro:if>
+    <xacro:unless value="${has_side_motion}">
+      <!-- Joint between the base and the ${prefix} upper leg -->
+      <joint name="${prefix}_hfe_joint" type="revolute">
+        <parent link="trunk"/>
+        <child link="${prefix}_upper_leg"/>
+        <limit effort="1000" lower="-10" upper="10" velocity="1000"/>
+        <!-- joints rotates around the y-axis -->
+        <axis xyz="0 1 0"/>
+        <!-- placement of the joint -->
+        <xacro:if value="${is_front}">
+          <xacro:unless value="${is_right}">
+            <origin xyz="${base_2_HFE_x} ${base_2_HFE_y} 0" rpy="0 0 0" />
+          </xacro:unless>
+          <xacro:if value="${is_right}">
+            <origin xyz="${base_2_HFE_x} ${-base_2_HFE_y} 0" rpy="0 0 0" />
+          </xacro:if>
+        </xacro:if>
+        <xacro:unless value="${is_front}">
+          <xacro:unless value="${is_right}">
+            <origin xyz="${-base_2_HFE_x} ${base_2_HFE_y} 0" rpy="0 0 0" />
+          </xacro:unless>
+          <xacro:if value="${is_right}">
+            <origin xyz="${-base_2_HFE_x} ${-base_2_HFE_y} 0" rpy="0 0 0" />
+          </xacro:if>
+        </xacro:unless>
+        <!-- pybullet simulation parameters -->
+        <dynamics damping="0.0" friction="0.0"/>
+      </joint>
+    </xacro:unless>
     <!-- UPPER LEG LINK -->
     <link name="${prefix}_upper_leg">

File: xacro/solo.urdf.xacro (robot description, xacro)
@@ -67,4 +67,5 @@
       is_front="true"
       is_right="false"
+      has_side_motion="false"
       color_name="${color_name}"
       color="${color}"
@@ -76,4 +77,5 @@
       is_front="true"
       is_right="true"
+      has_side_motion="false"
       color_name="${color_name}"
       color="${color}"
@@ -85,4 +87,5 @@
       is_front="false"
       is_right="false"
+      has_side_motion="false"
       color_name="${color_name}"
       color="${color}"
@@ -94,4 +97,5 @@
       is_front="false"
       is_right="true"
+      has_side_motion="false"
       color_name="${color_name}"
       color="${color}"

Commit message: fixed collision name

File: urdfs/leg.gazebo.xacro (robot description, xacro)
@@ -81,5 +81,5 @@
                                 <update_rate>250.0</update_rate>
                                 <contact>
-                                        <collision>${name}_lowerleg_fixed_joint_lump__${name}_foot_collision_1</collision>
+                                        <collision>${name}_lower_leg_fixed_joint_lump__${name}_foot_collision_1</collision>
                                 </contact>
                                 <!-- the sensor readings in terms of force torques are expressed in the lowerleg frame

Commit message: correction of a typo on contact sensor and changed mu

File: urdfs/leg.gazebo.xacro (robot description, xacro)
@@ -61,5 +61,5 @@
                 <update_rate>250.0</update_rate>
                 <contact>
-                  <collision>${name}_lowerleg_collision</collision>
+                  <collision>${name}_lower_leg_collision</collision>
                 </contact>
                 <!-- the sensor readings in terms of force torques are expressed in the lowerleg frame
@@ -73,13 +73,16 @@
                         <kp>1000000.0</kp>
                         <kd>100.0</kd>
-                        <mu1>1.0</mu1>
-                        <mu2>1.0</mu2>
+                        <mu1>0.8</mu1>
+                        <mu2>0.8</mu2>
                         <maxVel>1.0</maxVel>
                         <maxContacts>1</maxContacts>
                         <sensor name="${name}_foot_contact_sensor" type="contact">
                                 <always_on>true</always_on>
-                                <update_rate>250.0</update_rate>
+                                <update_rate>1000.0</update_rate>
                                 <contact>
-                                        <collision>${name}_lowerleg_fixed_joint_lump__${name}_foot_collision_1</collision>
+                                        <!-- this param is the most important: if wrong, contact sensor does not work
+                                        Since get the correct value is quite complex, convert the xacro to urdf to sdf
+                                        You can get it looking for "collision name"-->
+                                        <collision>${name}_lower_leg_fixed_joint_lump__${name}_foot_collision_1</collision>
                                 </contact>
                                 <!-- the sensor readings in terms of force torques are expressed in the lowerleg frame
@@ -87,5 +90,6 @@
                                 <plugin name="${name}_foot_bumper" filename="libgazebo_ros_bumper.so">
                                         <bumperTopicName>/solo/${name}_foot_bumper</bumperTopicName>
-                                        <robotNamespace>solo</robotNamespace>
+                                        <!--robotNamespace>solo</robotNamespace-->
+                                        <frameName>${name}_foot</frameName>
                                 </plugin>
                         </sensor>

Commit message: updated names

File: urdfs/leg.gazebo.xacro (robot description, xacro)
@@ -61,5 +61,5 @@
                 <update_rate>250.0</update_rate>
                 <contact>
-                  <collision>${name}_lower_leg_collision</collision>
+                  <collision>${name}_lowerleg_collision</collision>
                 </contact>
                 <!-- the sensor readings in terms of force torques are expressed in the lowerleg frame
@@ -81,5 +81,5 @@
                                 <update_rate>1000.0</update_rate>
                                 <contact>
-                                        <collision>${name}_lower_leg_fixed_joint_lump__${name}_foot_collision_1</collision>
+                                        <collision>${name}_lowerleg_fixed_joint_lump__${name}_foot_collision_1</collision>
                                 </contact>
                                 <!-- the sensor readings in terms of force torques are expressed in the lowerleg frame

File: urdfs/leg.xacro (robot description, xacro)
@@ -180,5 +180,5 @@
             <joint name="${prefix}_hfe_joint" type="revolute">
                 <parent link="${prefix}_hip_assembly"/>
-                <child link="${prefix}_upper_leg"/>
+                <child link="${prefix}_upperleg"/>
                 <!-- joints rotates around the y-axis -->
                 <axis xyz="0 1 0"/>
@@ -221,5 +221,5 @@
             <joint name="${prefix}_hfe_joint" type="revolute">
                 <parent link="trunk"/>
-                <child link="${prefix}_upper_leg"/>
+                <child link="${prefix}_upperleg"/>
                 <limit effort="1000" lower="-10" upper="10" velocity="1000"/>
                 <!-- joints rotates around the y-axis -->
@@ -247,5 +247,5 @@
         </xacro:unless>
         <!-- UPPER LEG LINK -->
-        <link name="${prefix}_upper_leg">
+        <link name="${prefix}_upperleg">
             <!-- UPPER LEG LINK INERTIAL -->
             <xacro:unless value="${is_right}">
@@ -307,6 +307,6 @@
         <!-- KFE JOINT: Joint between the upper leg and the lower leg -->
         <joint name="${prefix}_kfe_joint" type="revolute">
-            <parent link="${prefix}_upper_leg"/>
-            <child link="${prefix}_lower_leg"/>
+            <parent link="${prefix}_upperleg"/>
+            <child link="${prefix}_lowerleg"/>
             <!-- joints rotates around the y-axis -->
             <axis xyz="0 1 0"/>
@@ -344,5 +344,5 @@
         </joint>
         <!-- LOWERLEG -->
-        <link name="${prefix}_lower_leg">
+        <link name="${prefix}_lowerleg">
             <!-- LOWER LEG LINK INERTIAL -->
             <xacro:unless value="${is_right}">
@@ -404,5 +404,5 @@
         <!-- ANKLE: (Fixed) joint between the lower leg and the foot -->
         <joint name="${prefix}_ankle" type="fixed">
-            <parent link="${prefix}_lower_leg"/>
+            <parent link="${prefix}_lowerleg"/>
             <child link="${prefix}_foot"/>
             <!-- Joint placement -->
