Commit message: position, velocity and effort bounds corrected

File: urdfs/leg.xacro (robot description, xacro)
@@ -23,15 +23,18 @@
                 <parent link="trunk"/>
                 <child link="${prefix}_hip_assembly"/>
-                <limit effort="1000" lower="-10" upper="10" velocity="1000"/>
                 <!-- joints rotates around the x-axis -->
                 <axis xyz="1 0 0"/>
-                <!-- placement of the joint -->
+                <!-- limit and placement of the joint -->
                 <xacro:if value="${is_front}">
                     <xacro:unless value="${is_right}">
                         <!-- LF_HAA_JOINT -->
+                        <!-- lower=-75°, upper=140, velocity=555.5rpm (=5000rpm motor-side) -->
+                        <limit effort="1.2" lower="-1.30899694" upper="2.44346095" velocity="58.17764173"/>
                         <origin xyz="${base_2_HAA_x} ${base_2_HAA_y} 0" rpy="0 0 0" />
                     </xacro:unless>
                     <xacro:if value="${is_right}">
                         <!-- RF_HAA_JOINT -->
+                        <!-- lower=-140°, upper=75, velocity=555.5rpm (=5000rpm motor-side) -->
+                        <limit effort="1.2" lower="-2.44346095" upper="1.30899694" velocity="58.17764173"/>
                         <origin xyz="${base_2_HAA_x} ${-base_2_HAA_y} 0" rpy="0 0 0" />
                     </xacro:if>
@@ -40,8 +43,12 @@
                     <xacro:unless value="${is_right}">
                         <!-- LH_HAA_JOINT -->
+                        <!-- lower=-75°, upper=140, velocity=555.5rpm (=5000rpm motor-side) -->
+                        <limit effort="1.2" lower="-1.30899694" upper="2.44346095" velocity="58.17764173"/>
                         <origin xyz="${-base_2_HAA_x} ${base_2_HAA_y} 0" rpy="0 0 0" />
                     </xacro:unless>
                     <xacro:if value="${is_right}">
                         <!-- RH_HAA_JOINT -->
+                        <!-- lower=-140°, upper=75, velocity=555.5rpm (=5000rpm motor-side) -->
+                        <limit effort="1.2" lower="-2.44346095" upper="1.30899694" velocity="58.17764173"/>
                         <origin xyz="${-base_2_HAA_x} ${-base_2_HAA_y} 0" rpy="0 0 0" />
                     </xacro:if>
@@ -170,13 +177,34 @@
                 <parent link="${prefix}_hip_assembly"/>
                 <child link="${prefix}_upper_leg"/>
-                <limit effort="1000" lower="-10" upper="10" velocity="1000"/>
                 <!-- joints rotates around the y-axis -->
                 <axis xyz="0 1 0"/>
-                <!-- placement of the joint -->
-                <xacro:if value="${is_right}">
-                    <origin xyz="0 ${-HAA_2_HFE_y} 0" rpy="0 0 0" />
+                <!-- limit and placement of the joint -->
+                <xacro:if value="${is_front}">
+                    <xacro:unless value="${is_right}">
+                        <!-- LF_HFE_JOINT -->
+                        <!-- lower=-225°, upper=90°, velocity=555.5rpm (=5000rpm motor-side) -->
+                        <limit effort="1.2" lower="-3.92699082" upper="1.57079633" velocity="58.17764173"/>
+                        <origin xyz="0 ${HAA_2_HFE_y} 0" rpy="0 0 0" />
+                    </xacro:unless>
+                    <xacro:if value="${is_right}">
+                        <!-- RF_HFE_JOINT -->
+                        <!-- lower=-225°, upper=90°, velocity=555.5rpm (=5000rpm motor-side) -->
+                        <limit effort="1.2" lower="-3.92699082" upper="1.57079633" velocity="58.17764173"/>
+                        <origin xyz="0 ${-HAA_2_HFE_y} 0" rpy="0 0 0" />
+                    </xacro:if>
                 </xacro:if>
-                <xacro:unless value="${is_right}">
-                    <origin xyz="0 ${HAA_2_HFE_y} 0" rpy="0 0 0" />
+                <xacro:unless value="${is_front}">
+                    <xacro:unless value="${is_right}">
+                        <!-- LH_HFE_JOINT -->
+                        <!-- lower=-90°, upper=225°, velocity=555.5rpm (=5000rpm motor-side) -->
+                        <limit effort="1.2" lower="-1.57079633" upper="3.92699082" velocity="58.17764173"/>
+                        <origin xyz="0 ${HAA_2_HFE_y} 0" rpy="0 0 0" />
+                    </xacro:unless>
+                    <xacro:if value="${is_right}">
+                        <!-- RF_HFE_JOINT -->
+                        <!-- lower=-90°, upper=225°, velocity=555.5rpm (=5000rpm motor-side) -->
+                        <limit effort="1.2" lower="-1.57079633" upper="3.92699082" velocity="58.17764173"/>
+                        <origin xyz="0 ${-HAA_2_HFE_y} 0" rpy="0 0 0" />
+                    </xacro:if>
                 </xacro:unless>
                 <!-- pybullet simulation parameters -->
@@ -277,13 +305,18 @@
             <parent link="${prefix}_upper_leg"/>
             <child link="${prefix}_lower_leg"/>
-            <limit effort="1000" lower="-10" upper="10" velocity="1000"/>
             <!-- joints rotates around the y-axis -->
             <axis xyz="0 1 0"/>
-            <!-- placement of the joint -->
+            <!-- limit and placement of the joint -->
             <xacro:if value="${is_front}">
                 <xacro:unless value="${is_right}">
+                    <!-- LF_KFE JOINT -->
+                    <!-- lower=-370°, upper=370°, velocity=555.5rpm (=5000rpm motor-side) -->
+                    <limit effort="1.2" lower="-6.45771823" upper="6.45771823" velocity="58.17764173"/>
                     <origin xyz="0 ${HFE_2_KFE_y} ${-HFE_2_KFE_z}" rpy="0 0 0" />
                 </xacro:unless>
                 <xacro:if value="${is_right}">
+                    <!-- RF_KFE JOINT -->
+                    <!-- lower=-370°, upper=370°, velocity=555.5rpm (=5000rpm motor-side) -->
+                    <limit effort="1.2" lower="-6.45771823" upper="6.45771823" velocity="58.17764173"/>
                     <origin xyz="0 ${-HFE_2_KFE_y} ${-HFE_2_KFE_z}" rpy="0 0 0" />
                 </xacro:if>
@@ -291,7 +324,13 @@
             <xacro:unless value="${is_front}">
                 <xacro:unless value="${is_right}">
+                    <!-- LH_KFE JOINT -->
+                    <!-- lower=-370°, upper=370°, velocity=555.5rpm (=5000rpm motor-side) -->
+                    <limit effort="1.2" lower="-6.45771823" upper="6.45771823" velocity="58.17764173"/>
                     <origin xyz="0 ${HFE_2_KFE_y} ${-HFE_2_KFE_z}" rpy="0 0 0" />
                 </xacro:unless>
                 <xacro:if value="${is_right}">
+                    <!-- RH_KFE JOINT -->
+                    <!-- lower=-370°, upper=370°, velocity=555.5rpm (=5000rpm motor-side) -->
+                    <limit effort="1.2" lower="-6.45771823" upper="6.45771823" velocity="58.17764173"/>
                     <origin xyz="0 ${-HFE_2_KFE_y} ${-HFE_2_KFE_z}" rpy="0 0 0" />
                 </xacro:if>
@@ -316,5 +355,5 @@
                 <!-- Right lower leg inertia -->
                 <inertial>
-                <origin xyz="0.0 -0.00787644 -0.08928215" rpy="0 0 0" />
+                <origin xyz="0.0 0.00787644 -0.08928215" rpy="0 0 0" />
                 <mass value="0.03070001"/>
                 <inertia ixx="0.00012024" ixy="0.0"         ixz="0.0"
@@ -399,4 +438,5 @@
                 <geometry>
                     <mesh filename="package://solo_description/meshes/stl/with_foot/solo_foot.stl"/>
+                    <!-- sphere radius="0.01"/-->
                 </geometry>
                 <material name="${color_name}">

Commit message: max effort is passed as a variable

File: urdfs/leg.xacro (robot description, xacro)
@@ -14,4 +14,5 @@
     <xacro:property name="KFE_2_FOOT_y" value="${8.0 * 0.001}" />
     <xacro:property name="KFE_2_FOOT_z" value="${160.00 * 0.001}" />
+    <xacro:property name="MAX_TORQUE" value="$1.2">
     <!-- This macro has for purpose to define a leg -->
     <xacro:macro name="leg" params="prefix is_front is_right has_side_motion
@@ -30,5 +31,5 @@
                         <!-- LF_HAA_JOINT -->
                         <!-- lower=-75°, upper=140, velocity=555.5rpm (=5000rpm motor-side) -->
-                        <limit effort="1.2" lower="-1.30899694" upper="2.44346095" velocity="58.17764173"/>
+                        <limit effort="${MAX_TORQUE}" lower="-1.30899694" upper="2.44346095" velocity="58.17764173"/>
                         <origin xyz="${base_2_HAA_x} ${base_2_HAA_y} 0" rpy="0 0 0" />
                     </xacro:unless>
@@ -36,5 +37,5 @@
                         <!-- RF_HAA_JOINT -->
                         <!-- lower=-140°, upper=75, velocity=555.5rpm (=5000rpm motor-side) -->
-                        <limit effort="1.2" lower="-2.44346095" upper="1.30899694" velocity="58.17764173"/>
+                        <limit effort="${MAX_TORQUE}" lower="-2.44346095" upper="1.30899694" velocity="58.17764173"/>
                         <origin xyz="${base_2_HAA_x} ${-base_2_HAA_y} 0" rpy="0 0 0" />
                     </xacro:if>
@@ -44,5 +45,5 @@
                         <!-- LH_HAA_JOINT -->
                         <!-- lower=-75°, upper=140, velocity=555.5rpm (=5000rpm motor-side) -->
-                        <limit effort="1.2" lower="-1.30899694" upper="2.44346095" velocity="58.17764173"/>
+                        <limit effort="${MAX_TORQUE}" lower="-1.30899694" upper="2.44346095" velocity="58.17764173"/>
                         <origin xyz="${-base_2_HAA_x} ${base_2_HAA_y} 0" rpy="0 0 0" />
                     </xacro:unless>
@@ -50,5 +51,5 @@
                         <!-- RH_HAA_JOINT -->
                         <!-- lower=-140°, upper=75, velocity=555.5rpm (=5000rpm motor-side) -->
-                        <limit effort="1.2" lower="-2.44346095" upper="1.30899694" velocity="58.17764173"/>
+                        <limit effort="${MAX_TORQUE}" lower="-2.44346095" upper="1.30899694" velocity="58.17764173"/>
                         <origin xyz="${-base_2_HAA_x} ${-base_2_HAA_y} 0" rpy="0 0 0" />
                     </xacro:if>
@@ -184,5 +185,5 @@
                         <!-- LF_HFE_JOINT -->
                         <!-- lower=-225°, upper=90°, velocity=555.5rpm (=5000rpm motor-side) -->
-                        <limit effort="1.2" lower="-3.92699082" upper="1.57079633" velocity="58.17764173"/>
+                        <limit effort="${MAX_TORQUE}" lower="-3.92699082" upper="1.57079633" velocity="58.17764173"/>
                         <origin xyz="0 ${HAA_2_HFE_y} 0" rpy="0 0 0" />
                     </xacro:unless>
@@ -190,5 +191,5 @@
                         <!-- RF_HFE_JOINT -->
                         <!-- lower=-225°, upper=90°, velocity=555.5rpm (=5000rpm motor-side) -->
-                        <limit effort="1.2" lower="-3.92699082" upper="1.57079633" velocity="58.17764173"/>
+                        <limit effort="${MAX_TORQUE}" lower="-3.92699082" upper="1.57079633" velocity="58.17764173"/>
                         <origin xyz="0 ${-HAA_2_HFE_y} 0" rpy="0 0 0" />
                     </xacro:if>
@@ -198,5 +199,5 @@
                         <!-- LH_HFE_JOINT -->
                         <!-- lower=-90°, upper=225°, velocity=555.5rpm (=5000rpm motor-side) -->
-                        <limit effort="1.2" lower="-1.57079633" upper="3.92699082" velocity="58.17764173"/>
+                        <limit effort="${MAX_TORQUE}" lower="-1.57079633" upper="3.92699082" velocity="58.17764173"/>
                         <origin xyz="0 ${HAA_2_HFE_y} 0" rpy="0 0 0" />
                     </xacro:unless>
@@ -204,5 +205,5 @@
                         <!-- RF_HFE_JOINT -->
                         <!-- lower=-90°, upper=225°, velocity=555.5rpm (=5000rpm motor-side) -->
-                        <limit effort="1.2" lower="-1.57079633" upper="3.92699082" velocity="58.17764173"/>
+                        <limit effort="${MAX_TORQUE}" lower="-1.57079633" upper="3.92699082" velocity="58.17764173"/>
                         <origin xyz="0 ${-HAA_2_HFE_y} 0" rpy="0 0 0" />
                     </xacro:if>
@@ -312,5 +313,5 @@
                     <!-- LF_KFE JOINT -->
                     <!-- lower=-370°, upper=370°, velocity=555.5rpm (=5000rpm motor-side) -->
-                    <limit effort="1.2" lower="-6.45771823" upper="6.45771823" velocity="58.17764173"/>
+                    <limit effort="${MAX_TORQUE}" lower="-6.45771823" upper="6.45771823" velocity="58.17764173"/>
                     <origin xyz="0 ${HFE_2_KFE_y} ${-HFE_2_KFE_z}" rpy="0 0 0" />
                 </xacro:unless>
@@ -318,5 +319,5 @@
                     <!-- RF_KFE JOINT -->
                     <!-- lower=-370°, upper=370°, velocity=555.5rpm (=5000rpm motor-side) -->
-                    <limit effort="1.2" lower="-6.45771823" upper="6.45771823" velocity="58.17764173"/>
+                    <limit effort="${MAX_TORQUE}" lower="-6.45771823" upper="6.45771823" velocity="58.17764173"/>
                     <origin xyz="0 ${-HFE_2_KFE_y} ${-HFE_2_KFE_z}" rpy="0 0 0" />
                 </xacro:if>
@@ -326,5 +327,5 @@
                     <!-- LH_KFE JOINT -->
                     <!-- lower=-370°, upper=370°, velocity=555.5rpm (=5000rpm motor-side) -->
-                    <limit effort="1.2" lower="-6.45771823" upper="6.45771823" velocity="58.17764173"/>
+                    <limit effort="${MAX_TORQUE}" lower="-6.45771823" upper="6.45771823" velocity="58.17764173"/>
                     <origin xyz="0 ${HFE_2_KFE_y} ${-HFE_2_KFE_z}" rpy="0 0 0" />
                 </xacro:unless>
@@ -332,5 +333,5 @@
                     <!-- RH_KFE JOINT -->
                     <!-- lower=-370°, upper=370°, velocity=555.5rpm (=5000rpm motor-side) -->
-                    <limit effort="1.2" lower="-6.45771823" upper="6.45771823" velocity="58.17764173"/>
+                    <limit effort="${MAX_TORQUE}" lower="-6.45771823" upper="6.45771823" velocity="58.17764173"/>
                     <origin xyz="0 ${-HFE_2_KFE_y} ${-HFE_2_KFE_z}" rpy="0 0 0" />
                 </xacro:if>

Commit message: typo correction in max torque value

File: urdfs/leg.xacro (robot description, xacro)
@@ -14,5 +14,5 @@
     <xacro:property name="KFE_2_FOOT_y" value="${8.0 * 0.001}" />
     <xacro:property name="KFE_2_FOOT_z" value="${160.00 * 0.001}" />
-    <xacro:property name="MAX_TORQUE" value="$1.2">
+    <xacro:property name="MAX_TORQUE" value="1.2" />
     <!-- This macro has for purpose to define a leg -->
     <xacro:macro name="leg" params="prefix is_front is_right has_side_motion

Commit message: gear_ratio, motor_Kt, max_curr added as xacro properties

File: urdfs/leg.xacro (robot description, xacro)
@@ -14,5 +14,8 @@
     <xacro:property name="KFE_2_FOOT_y" value="${8.0 * 0.001}" />
     <xacro:property name="KFE_2_FOOT_z" value="${160.00 * 0.001}" />
-    <xacro:property name="MAX_TORQUE" value="1.2" />
+    <xacro:property name="gear_ratio" value="9.0" />
+    <xacro:property name="motor_Kt"   value="0.025" />
+    <xacro:property name="max_curr"   value="7.0" />
+    <xacro:property name="MAX_TORQUE" value="${gear_ratio * motor_Kt * max_curr}" />
     <!-- This macro has for purpose to define a leg -->
     <xacro:macro name="leg" params="prefix is_front is_right has_side_motion

Commit message: renaming link to be consistent with aliengo and go1

File: urdfs/leg.xacro (robot description, xacro)
@@ -26,5 +26,5 @@
             <joint name="${prefix}_haa_joint" type="revolute">
                 <parent link="trunk"/>
-                <child link="${prefix}_hip_assembly"/>
+                <child link="${prefix}_hip"/>
                 <!-- joints rotates around the x-axis -->
                 <axis xyz="1 0 0"/>
@@ -62,5 +62,5 @@
             </joint>
             <!-- HIP ASSEMBLY -->
-            <link name="${prefix}_hip_assembly">
+            <link name="${prefix}_hip">
             	<!-- create a dummy hip_assembly link to join the two joints -->
             	<!-- HIP ASSEMBLY VISUAL-->
@@ -179,5 +179,5 @@
             <!--HFE JOINT-->
             <joint name="${prefix}_hfe_joint" type="revolute">
-                <parent link="${prefix}_hip_assembly"/>
+                <parent link="${prefix}_hip"/>
                 <child link="${prefix}_upperleg"/>
                 <!-- joints rotates around the y-axis -->
