Commit message: Add flywheels in srdf.xacro and indentation modification

File: robots/solo.srdf.xacro (robot description, xacro)
@@ -1,37 +1,106 @@
+<?xml version="1.0" ?>
 <robot name="solo" xmlns:xacro="http://ros.org/wiki/xacro">
-  <group name="base">
-    <link name="base_link"/>
-  </group>
-  <group name="lf">
-    <chain base_link="trunk" tip_link="lf_foot"/>
-  </group>
-  <group name="rf">
-    <chain base_link="trunk" tip_link="rf_foot"/>
-  </group>
-  <group name="lh">
-    <chain base_link="trunk" tip_link="lh_foot"/>
-  </group>
-  <group name="rh">
-    <chain base_link="trunk" tip_link="rh_foot"/>
-  </group>
-  <group name="chains">
-    <group name="lf"/>
-    <group name="rf"/>
-    <group name="lh"/>
-    <group name="rh"/>
-  </group>
-  <group_state group="chains" name="home">
-    <joint name="lf_haa_joint" value="-0.2"/>
-    <joint name="lf_hfe_joint" value="0.75"/>
-    <joint name="lf_kfe_joint" value="-1.5"/>
-    <joint name="rf_haa_joint" value="-0.2"/>
-    <joint name="rf_hfe_joint" value="0.75"/>
-    <joint name="rf_kfe_joint" value="-1.5"/>
-    <joint name="lh_haa_joint" value="-0.2"/>
-    <joint name="lh_hfe_joint" value="0.75"/>
-    <joint name="lh_kfe_joint" value="-1.5"/>
-    <joint name="rh_haa_joint" value="-0.2"/>
-    <joint name="rh_hfe_joint" value="0.75"/>
-    <joint name="rh_kfe_joint" value="-1.5"/>
-  </group_state>
+	<xacro:arg name="flywheel" default="false"/>
+    <!-- left front leg -->
+    <group name="lf_leg">
+        <joint name="lf_haa_joint" />
+        <joint name="lf_hfe_joint" />
+        <joint name="lf_kfe_joint" />
+        <chain base_link="base_link" tip_link="lf_foot" />
+    </group>
+    <!-- right front leg -->
+    <group name="rf_leg">
+        <joint name="rf_haa_joint" />
+        <joint name="rf_hfe_joint" />
+        <joint name="rf_kfe_joint" />
+        <chain base_link="base_link" tip_link="rf_foot" />
+    </group>
+    <!-- left hind leg -->
+    <group name="lh_leg">
+        <joint name="lh_haa_joint" />
+        <joint name="lh_hfe_joint" />
+        <joint name="lh_kfe_joint" />
+        <chain base_link="base_link" tip_link="lh_foot" />
+    </group>
+    <!-- right hind leg -->
+    <group name="rh_leg">
+        <joint name="rh_haa_joint" />
+        <joint name="rh_hfe_joint" />
+        <joint name="rh_kfe_joint" />
+        <chain base_link="base_link" tip_link="rh_foot" />
+    </group>
+    <end_effector name="lf_foot" parent_link="FL_FOOT" group="lf_leg" />
+    <end_effector name="rf_foot" parent_link="FR_FOOT" group="rf_leg" />
+    <end_effector name="lh_foot" parent_link="HL_FOOT" group="lh_leg" />
+    <end_effector name="rh_foot" parent_link="HR_FOOT" group="rh_leg" />
+    <!-- Include flywheel -->
+	<xacro:if value="$(arg flywheel)">
+	    <group name="l_wheel">
+		    <joint name="z_left_wheel_joint" />
+    	</group>
+    	<group name="r_wheel">
+		    <joint name="z_right_wheel_joint" />
+    	</group>
+    	<group name="f_wheel">
+		    <joint name="z_front_wheel_joint" />
+    	</group>
+    	<group name="b_wheel">
+		    <joint name="z_back_wheel_joint" />
+    	</group>
+		<group name="flywheel">
+		    <group name="l_wheel" />
+		    <group name="r_wheel" />
+		    <group name="f_wheel" />
+		    <group name="b_wheel" />
+		</group>
+		<group name="all_legs_and_flywheel">
+		    <group name="lf" />
+		    <group name="rf" />
+		    <group name="lh" />
+		    <group name="rh" />
+		    <group name="flywheel" />
+		</group>
+		<group_state name="standing" group="all_legs">
+		    <joint name="floating_base_joint" value="0. 0. 0.223 0. 0. 0. 1." />
+		    <joint name="lf_haa_joint" value="-0.2" />
+		    <joint name="lf_hfe_joint" value="0.78539816" />
+		    <joint name="lf_kfe_joint" value="-1.57079633" />
+		    <joint name="lh_haa_joint" value="-0.2" />
+		    <joint name="lh_hfe_joint" value="-0.78539816" />
+		    <joint name="lh_kfe_joint" value="1.57079633" />
+		    <joint name="rf_haa_joint" value="-0.2" />
+		    <joint name="rf_hfe_joint" value="0.78539816" />
+		    <joint name="rf_kfe_joint" value="-1.57079633" />
+		    <joint name="rh_haa_joint" value="-0.2" />
+		    <joint name="rh_hfe_joint" value="-0.78539816" />
+		    <joint name="rh_kfe_joint" value="1.57079633" />
+		    <joint name="z_left_wheel_joint"  value="0" />
+		    <joint name="z_right_wheel_joint" value="0" />
+		    <joint name="z_front_wheel_joint" value="0" />
+		    <joint name="z_back_wheel_joint"  value="0" />
+		</group_state>
+	</xacro:if>
+	<xacro:unless value="$(arg flywheel)">
+		<group name="all_legs">
+		    <group name="lf" />
+		    <group name="rf" />
+		    <group name="lh" />
+		    <group name="rh" />
+		</group>
+		<group_state name="standing" group="all_legs">
+		    <joint name="floating_base_joint" value="0. 0. 0.223 0. 0. 0. 1." />
+		    <joint name="lf_haa_joint" value="-0.2" />
+		    <joint name="lf_hfe_joint" value="0.78539816" />
+		    <joint name="lf_kfe_joint" value="-1.57079633" />
+		    <joint name="lh_haa_joint" value="-0.2" />
+		    <joint name="lh_hfe_joint" value="-0.78539816" />
+		    <joint name="lh_kfe_joint" value="1.57079633" />
+		    <joint name="rf_haa_joint" value="-0.2" />
+		    <joint name="rf_hfe_joint" value="0.78539816" />
+		    <joint name="rf_kfe_joint" value="-1.57079633" />
+		    <joint name="rh_haa_joint" value="-0.2" />
+		    <joint name="rh_hfe_joint" value="-0.78539816" />
+		    <joint name="rh_kfe_joint" value="1.57079633" />
+		</group_state>
+	</xacro:unless>
 </robot>

File: robots/solo.urdf.xacro (robot description, xacro)
@@ -1,108 +1,110 @@
 <?xml version="1.0" ?>
 <robot name="solo" xmlns:xacro="http://ros.org/wiki/xacro">
-  <xacro:property name="color_name" value="grey" />
-  <xacro:property name="color" value="0.8 0.8 0.8" />
-  <xacro:property name="opacity" value="1.0" />
-  <xacro:arg name="flywheel" default="false"/>
-  <xacro:arg name="load_force_sensors" default="false"/>
-  <xacro:arg name="new_gazebo_version" default="false"/>
-        <xacro:include filename="$(find solo_description)/gazebo/gazebo.urdf.xacro">
-             <xacro:arg name="task_period" value="$(arg task_period)"/>
-        </xacro:include>
-	     <xacro:unless value="$(arg new_gazebo_version)">
-		        <!-- Floating-base Joint -->
-		        <link name="world"/>
-		        <joint name="floating_base_joint" type="floating" >
-		            <origin rpy="0 0 0" xyz="0 0 0"/>
-		            <parent link="world"/>
-		            <child link="base_link"/>
-		        </joint>
-	     </xacro:unless>
-	     	<link name="base_link" />
-		        <joint name="floating_base" type="fixed">
-		            <origin rpy="0 0 0" xyz="0 0 0"/>
-		            <parent link="base_link"/>
-		            <child link="trunk"/>
-		</joint>
-		<link name="trunk">
-			<inertial>
-			    <origin xyz="0 0 0" rpy="0 0 0" />
-			    <mass value="1.63315091"/>
-			    <!-- The base is extremely symmetrical. -->
-			    <inertia ixx="0.00578574" ixy="0.0" ixz="0.0"
-				                      iyy="0.01938108" iyz="0.0"
-				                                       izz="0.02476124"/>
-			</inertial>
-			<visual>
-				<origin xyz="0 0 0" rpy="0 0 0" />
-				    <geometry>
-				      <mesh filename="package://solo_description/meshes/stl/with_foot/solo_body.stl"/>
-				    </geometry>
-                                    <material name="${color_name}">
-				        <color rgba="${color} ${opacity}"/>
-				    </material>
-			</visual>
-			<collision>
-		            <origin xyz="0 0 0" rpy="0 0 0" />
-		            <geometry>
-		              <mesh filename="package://solo_description/meshes/stl/with_foot/solo_body.stl"/>
-		            </geometry>
-		            <material name="${color_name}">
-		                <color rgba="${color} ${opacity}"/>
-		            </material>
-               		 </collision>
-			<!-- Bullet specific paramters -->
-		        <contact>
-		          <lateral_friction value="1.0"/>
-		          <restitution value="0.5"/>
-		        </contact>
-		</link>
- 	 <!-- Include the legs -->
-  	<xacro:include filename="$(find solo_description)/urdfs/leg.xacro"/>
-        <!-- Include flywheel -->
-        <xacro:if value="$(arg flywheel)">
-              <xacro:include filename="$(find solo_description)/urdfs/flywheel.xacro"/>
-              <!-- inertia =  m*radius^2 but I had to set 10 times more for sm stability-->
-              <xacro:flywheel_train radius="0.05" mass_lr="0.1" inertia_lr="0.00025"  mass_fh="0.1" inertia_fh="0.00025"/>
-        </xacro:if>
-  <!-- Include the front left leg -->
-  <xacro:leg
-      prefix="lf"
-      is_front="true"
-      is_right="false"
-      has_side_motion="true"
-      color_name="${color_name}"
-      color="${color}"
-      opacity="${opacity}"
-      load_force_sensors="$(arg load_force_sensors)"/>
-  <!-- Include the front right leg -->
-  <xacro:leg
-      prefix="rf"
-      is_front="true"
-      is_right="true"
-      has_side_motion="true"
-      color_name="${color_name}"
-      color="${color}"
-      opacity="${opacity}"
-      load_force_sensors="$(arg load_force_sensors)"/>
-  <!-- Include the hind left leg -->
-  <xacro:leg
-      prefix="lh"
-      is_front="false"
-      is_right="false"
-      has_side_motion="true"
-      color_name="${color_name}"
-      color="${color}"
-      opacity="${opacity}"
-      load_force_sensors="$(arg load_force_sensors)"/>
-  <!-- Include the hind right leg -->
-  <xacro:leg
-      prefix="rh"
-      is_front="false"
-      is_right="true"
-      has_side_motion="true"
-      color_name="${color_name}"
-      color="${color}"
-      opacity="${opacity}"
-      load_force_sensors="$(arg load_force_sensors)"/>
+    <xacro:property name="color_name" value="grey" />
+    <xacro:property name="color" value="0.8 0.8 0.8" />
+    <xacro:property name="opacity" value="1.0" />
+    <xacro:arg name="flywheel" default="false"/>
+    <xacro:arg name="load_force_sensors" default="false"/>
+    <xacro:arg name="new_gazebo_version" default="true"/>
+    <xacro:include filename="$(find solo_description)/gazebo/gazebo.urdf.xacro">
+         <xacro:arg name="task_period" value="$(arg task_period)"/>
+    </xacro:include>
+    <!-- BASE LINK -->
+    <!-- floating type is supported in older versions of Gazebo. In new Gazebo if a link has no parent, it is supposed to be attached to a floating joint -->
+    <xacro:unless value="$(arg new_gazebo_version)">
+        <!-- Floating-base Joint -->
+        <link name="world"/>
+        <joint name="floating_base_joint" type="floating" >
+            <origin rpy="0 0 0" xyz="0 0 0"/>
+            <parent link="world"/>
+            <child link="base_link"/>
+        </joint>
+    </xacro:unless>
+    <link name="base_link" />
+    <joint name="floating_base" type="fixed">
+        <origin rpy="0 0 0" xyz="0 0 0"/>
+        <parent link="base_link"/>
+        <child link="trunk"/>
+    </joint>
+    <link name="trunk">
+        <inertial>
+            <origin xyz="0 0 0" rpy="0 0 0" />
+            <mass value="1.16115091"/>
+            <!-- The base is extremely symmetrical. -->
+            <inertia ixx="0.00578574" ixy="0.0"        ixz="0.0"
+                                      iyy="0.01938108" iyz="0.0"
+                                                       izz="0.02476124"/>
+        </inertial>
+        <visual>
+            <origin xyz="0 0 0" rpy="0 0 0" />
+            <geometry>
+                <mesh filename="package://solo_description/meshes/stl/with_foot/solo_body.stl"/>
+            </geometry>
+            <material name="${color_name}">
+                <color rgba="${color} ${opacity}"/>
+            </material>
+        </visual>
+        <collision>
+            <origin xyz="0 0 0" rpy="0 0 0" />
+            <geometry>
+                <mesh filename="package://solo_description/meshes/stl/with_foot/solo_body.stl"/>
+            </geometry>
+            <material name="${color_name}">
+                <color rgba="${color} ${opacity}"/>
+            </material>
+        </collision>
+        <!-- Bullet specific paramters -->
+        <contact>
+        <lateral_friction value="1.0"/>
+        <restitution value="0.5"/>
+        </contact>
+    </link>
+    <!-- Include legs -->
+    <xacro:include filename="$(find solo_description)/urdfs/leg.xacro"/>
+    <!-- Include flywheels -->
+    <xacro:if value="$(arg flywheel)">
+          <xacro:include filename="$(find solo_description)/urdfs/flywheel.xacro"/>
+          <!-- inertia =  m*radius^2 but I had to set 10 times more for sm stability-->
+          <xacro:flywheel_train radius="0.05" mass_lr="0.1" inertia_lr="0.00025"  mass_fh="0.1" inertia_fh="0.00025"/>
+    </xacro:if>
+    <!-- LEFT FRONT LEG -->
+    <xacro:leg
+        prefix="lf"
+        is_front="true"
+        is_right="false"
+        has_side_motion="true"
+        color_name="${color_name}"
+        color="${color}"
+        opacity="${opacity}"
+        load_force_sensors="$(arg load_force_sensors)"/>
+    <!-- RIGHT FRONT LEG -->
+    <xacro:leg
+        prefix="rf"
+        is_front="true"
+        is_right="true"
+        has_side_motion="true"
+        color_name="${color_name}"
+        color="${color}"
+        opacity="${opacity}"
+        load_force_sensors="$(arg load_force_sensors)"/>
+    <!-- LEFT HIND LEG -->
+    <xacro:leg
+        prefix="lh"
+        is_front="false"
+        is_right="false"
+        has_side_motion="true"
+        color_name="${color_name}"
+        color="${color}"
+        opacity="${opacity}"
+        load_force_sensors="$(arg load_force_sensors)"/>
+    <!-- RIGHT HIND LEG -->
+    <xacro:leg
+        prefix="rh"
+        is_front="false"
+        is_right="true"
+        has_side_motion="true"
+        color_name="${color_name}"
+        color="${color}"
+        opacity="${opacity}"
+        load_force_sensors="$(arg load_force_sensors)"/>
 </robot>

Commit message: using srdf for go0 (need to install ros_kinetic_srdfdom)

File: robots/solo.srdf.xacro (robot description, xacro)
@@ -61,18 +61,18 @@
 		    <group name="flywheel" />
 		</group>
-		<group_state name="standing" group="all_legs">
+                <group_state name="home" group="all_legs">
 		    <joint name="floating_base_joint" value="0. 0. 0.223 0. 0. 0. 1." />
 		    <joint name="lf_haa_joint" value="-0.2" />
-		    <joint name="lf_hfe_joint" value="0.78539816" />
-		    <joint name="lf_kfe_joint" value="-1.57079633" />
+                    <joint name="lf_hfe_joint" value="0.75" />
+                    <joint name="lf_kfe_joint" value="-1.5" />
 		    <joint name="lh_haa_joint" value="-0.2" />
-		    <joint name="lh_hfe_joint" value="-0.78539816" />
-		    <joint name="lh_kfe_joint" value="1.57079633" />
+                    <joint name="lh_hfe_joint" value="-0.75" />
+                    <joint name="lh_kfe_joint" value="1.5" />
 		    <joint name="rf_haa_joint" value="-0.2" />
-		    <joint name="rf_hfe_joint" value="0.78539816" />
-		    <joint name="rf_kfe_joint" value="-1.57079633" />
+                    <joint name="rf_hfe_joint" value="0.75" />
+                    <joint name="rf_kfe_joint" value="-1.5" />
 		    <joint name="rh_haa_joint" value="-0.2" />
-		    <joint name="rh_hfe_joint" value="-0.78539816" />
-		    <joint name="rh_kfe_joint" value="1.57079633" />
+                    <joint name="rh_hfe_joint" value="-0.75" />
+                    <joint name="rh_kfe_joint" value="1.5" />
 		    <joint name="z_left_wheel_joint"  value="0" />
 		    <joint name="z_right_wheel_joint" value="0" />
@@ -88,18 +88,18 @@
 		    <group name="rh" />
 		</group>
-		<group_state name="standing" group="all_legs">
+                <group_state name="home" group="all_legs">
 		    <joint name="floating_base_joint" value="0. 0. 0.223 0. 0. 0. 1." />
-		    <joint name="lf_haa_joint" value="-0.2" />
-		    <joint name="lf_hfe_joint" value="0.78539816" />
-		    <joint name="lf_kfe_joint" value="-1.57079633" />
-		    <joint name="lh_haa_joint" value="-0.2" />
-		    <joint name="lh_hfe_joint" value="-0.78539816" />
-		    <joint name="lh_kfe_joint" value="1.57079633" />
-		    <joint name="rf_haa_joint" value="-0.2" />
-		    <joint name="rf_hfe_joint" value="0.78539816" />
-		    <joint name="rf_kfe_joint" value="-1.57079633" />
-		    <joint name="rh_haa_joint" value="-0.2" />
-		    <joint name="rh_hfe_joint" value="-0.78539816" />
-		    <joint name="rh_kfe_joint" value="1.57079633" />
+                    <joint name="lf_haa_joint" value="0.2" />
+                    <joint name="lf_hfe_joint" value="0.75" />
+                    <joint name="lf_kfe_joint" value="-1.5" />
+                    <joint name="lh_haa_joint" value="0.2" />
+                    <joint name="lh_hfe_joint" value="-0.75" />
+                    <joint name="lh_kfe_joint" value="1.5" />
+                    <joint name="rf_haa_joint" value="-0.2" />
+                    <joint name="rf_hfe_joint" value="0.75" />
+                    <joint name="rf_kfe_joint" value="-1.5" />
+                    <joint name="rh_haa_joint" value="-0.2" />
+                    <joint name="rh_hfe_joint" value="-0.75" />
+                    <joint name="rh_kfe_joint" value="1.5" />
 		</group_state>
 	</xacro:unless>

Commit message: changed intial position put zero on haa
Signed-off-by: Andrea Cumerlotti <andrea.cumerlotti@iit.it>

File: robots/solo.srdf.xacro (robot description, xacro)
@@ -63,14 +63,14 @@
                 <group_state name="home" group="all_legs">
 		    <joint name="floating_base_joint" value="0. 0. 0.223 0. 0. 0. 1." />
-		    <joint name="lf_haa_joint" value="-0.2" />
+		    <joint name="lf_haa_joint" value="-0.0" />
                     <joint name="lf_hfe_joint" value="0.75" />
                     <joint name="lf_kfe_joint" value="-1.5" />
-		    <joint name="lh_haa_joint" value="-0.2" />
+		    <joint name="lh_haa_joint" value="-0.0" />
                     <joint name="lh_hfe_joint" value="-0.75" />
                     <joint name="lh_kfe_joint" value="1.5" />
-		    <joint name="rf_haa_joint" value="-0.2" />
+		    <joint name="rf_haa_joint" value="-0.0" />
                     <joint name="rf_hfe_joint" value="0.75" />
                     <joint name="rf_kfe_joint" value="-1.5" />
-		    <joint name="rh_haa_joint" value="-0.2" />
+		    <joint name="rh_haa_joint" value="-0.0" />
                     <joint name="rh_hfe_joint" value="-0.75" />
                     <joint name="rh_kfe_joint" value="1.5" />
@@ -90,14 +90,14 @@
                 <group_state name="home" group="all_legs">
 		    <joint name="floating_base_joint" value="0. 0. 0.223 0. 0. 0. 1." />
-                    <joint name="lf_haa_joint" value="0.2" />
+                    <joint name="lf_haa_joint" value="0.0" />
                     <joint name="lf_hfe_joint" value="0.75" />
                     <joint name="lf_kfe_joint" value="-1.5" />
-                    <joint name="lh_haa_joint" value="0.2" />
+                    <joint name="lh_haa_joint" value="0.0" />
                     <joint name="lh_hfe_joint" value="-0.75" />
                     <joint name="lh_kfe_joint" value="1.5" />
-                    <joint name="rf_haa_joint" value="-0.2" />
+                    <joint name="rf_haa_joint" value="-0.0" />
                     <joint name="rf_hfe_joint" value="0.75" />
                     <joint name="rf_kfe_joint" value="-1.5" />
-                    <joint name="rh_haa_joint" value="-0.2" />
+                    <joint name="rh_haa_joint" value="-0.0" />
                     <joint name="rh_hfe_joint" value="-0.75" />
                     <joint name="rh_kfe_joint" value="1.5" />
