Commit message: [important!] renamed folder xacro into robots
renamed fly into flywheel param

File: robots/solo.urdf.xacro (robot description, xacro)
@@ -5,5 +5,5 @@
   xmlns:sensor="http://playerstage.sourceforge.net/gazebo/xmlschema/#sensor"
   xmlns:xacro="http://ros.org/wiki/xacro">
-  <xacro:arg name="fly" default="false"/>
+  <xacro:arg name="flywheel" default="false"/>
   <xacro:arg name="load_force_sensors" default="false"/>
   <xacro:property name="color_name" value="grey" />
@@ -62,7 +62,7 @@
   	<xacro:include filename="$(find solo_description)/urdfs/leg.xacro"/>
         <!-- Include flywheel -->
-        <xacro:if value="$(arg fly)">
+        <xacro:if value="$(arg flywheel)">
               <xacro:include filename="$(find solo_description)/urdfs/flywheel.xacro"/>
-                 <xacro:flywheel_train radius="0.05" />
+              <xacro:flywheel_train radius="0.05" mass_lr="0.2" inertia_lr="0.1"  mass_fh="0.2" inertia_fh="0.1"/>
         </xacro:if>
   <!-- Include the front left leg -->

File: urdfs/flywheel.xacro (robot description, xacro)
@@ -2,5 +2,5 @@
 <robot xmlns:xacro="http://ros.org/wiki/xacro" name="solo">
 <!-- Things that are needed only for Gazebo (not the physical robot). These include sensor and controller plugin specifications -->
-<xacro:macro name="flywheel_train" params="radius">
+<xacro:macro name="flywheel_train" params="radius mass_fh mass_lr inertia_fh inertia_lr">
     <xacro:include filename="$(find solo_description)/urdfs/flywheel.transmission.xacro"/>
     <xacro:include filename="$(find solo_description)/urdfs/flywheel.gazebo.xacro"/>
@@ -14,6 +14,6 @@
     <link name="left_wheel">
     <inertial>
-    <mass value="0.2"/>
-    <inertia ixx="0.001" ixy="0" ixz="0" iyy="0.001" iyz="0" izz="0.001"/>
+    <mass value="${mass_lr}"/>
+    <inertia ixx="0.001" ixy="0" ixz="0" iyy="0.001" iyz="0" izz="${inertia_lr}"/>
     </inertial>
     <visual>
@@ -38,6 +38,6 @@
     <link name="right_wheel">
     <inertial>
-    <mass value="0.2"/>
-    <inertia ixx="0.001" ixy="0" ixz="0" iyy="0.001" iyz="0" izz="0.001"/>
+    <mass value="${mass_lr}"/>
+    <inertia ixx="0.001" ixy="0" ixz="0" iyy="0.001" iyz="0" izz="${inertia_lr}"/>
     </inertial>
     <visual>
@@ -63,6 +63,6 @@
     <link name="front_wheel">
     <inertial>
-    <mass value="0.2"/>
-    <inertia ixx="0.001" ixy="0" ixz="0" iyy="0.001" iyz="0" izz="0.001"/>
+    <mass value="${mass_fh}"/>
+    <inertia ixx="0.001" ixy="0" ixz="0" iyy="0.001" iyz="0" izz="${inertia_fh}"/>
     </inertial>
     <visual>
@@ -88,6 +88,6 @@
     <link name="back_wheel">
         <inertial>
-        <mass value="0.2"/>
-        <inertia ixx="0.001" ixy="0" ixz="0" iyy="0.001" iyz="0" izz="0.001"/>
+        <mass value="${mass_fh}"/>
+        <inertia ixx="0.001" ixy="0" ixz="0" iyy="0.001" iyz="0" izz="${inertia_fh}"/>
         </inertial>
         <visual>

Commit message: parametryzing inertian in flywheel
setting revolute joints cause continuous create issues in Pinocchio (2
joints)
setting flywheel as an external input parameter

File: robots/solo.urdf.xacro (robot description, xacro)
@@ -1,13 +1,9 @@
 <?xml version="1.0" ?>
-<robot name="solo"
-  xmlns:controller="http://playerstage.sourceforge.net/gazebo/xmlschema/#controller"
-  xmlns:interface="http://ros.org/wiki/xacro"
-  xmlns:sensor="http://playerstage.sourceforge.net/gazebo/xmlschema/#sensor"
-  xmlns:xacro="http://ros.org/wiki/xacro">
-  <xacro:arg name="flywheel" default="false"/>
-  <xacro:arg name="load_force_sensors" default="false"/>
+<robot name="solo" xmlns:xacro="http://ros.org/wiki/xacro">
   <xacro:property name="color_name" value="grey" />
   <xacro:property name="color" value="0.8 0.8 0.8" />
   <xacro:property name="opacity" value="1.0" />
+  <xacro:arg name="flywheel" default="false"/>
+  <xacro:arg name="load_force_sensors" default="false"/>
         <xacro:include filename="$(find solo_description)/gazebo/gazebo.urdf.xacro">
              <xacro:arg name="task_period" value="$(arg task_period)"/>
@@ -64,5 +60,6 @@
         <xacro:if value="$(arg flywheel)">
               <xacro:include filename="$(find solo_description)/urdfs/flywheel.xacro"/>
-              <xacro:flywheel_train radius="0.05" mass_lr="0.2" inertia_lr="0.1"  mass_fh="0.2" inertia_fh="0.1"/>
+              <!-- inertia = 0.5 m*radius^2 but I had to set 10 times more for sm stability-->
+              <xacro:flywheel_train radius="0.05" mass_lr="0.2" inertia_lr="0.0025"  mass_fh="0.2" inertia_fh="0.0025"/>
         </xacro:if>
   <!-- Include the front left leg -->

File: urdfs/flywheel.transmission.xacro (robot description, xacro)
@@ -5,8 +5,8 @@
             <type>transmission_interface/SimpleTransmission</type>
             <joint name="z_right_wheel_joint">
-                    <hardwareInterface>EffortJointInterface</hardwareInterface>
+                    <hardwareInterface>hardware_interface/EffortJointInterface</hardwareInterface>
             </joint>
             <actuator name="z_right_wheel_motor">
-                    <hardwareInterface>EffortJointInterface</hardwareInterface>
+                    <hardwareInterface>hardware_interface/EffortJointInterface</hardwareInterface>
                     <mechanicalReduction>1</mechanicalReduction>
             </actuator>
@@ -15,8 +15,8 @@
             <type>transmission_interface/SimpleTransmission</type>
             <joint name="z_left_wheel_joint">
-                    <hardwareInterface>EffortJointInterface</hardwareInterface>
+                    <hardwareInterface>hardware_interface/EffortJointInterface</hardwareInterface>
             </joint>
             <actuator name="z_left_wheel_motor">
-                    <hardwareInterface>EffortJointInterface</hardwareInterface>
+                    <hardwareInterface>hardware_interface/EffortJointInterface</hardwareInterface>
                     <mechanicalReduction>1</mechanicalReduction>
             </actuator>
@@ -25,8 +25,8 @@
             <type>transmission_interface/SimpleTransmission</type>
             <joint name="z_back_wheel_joint">
-                    <hardwareInterface>EffortJointInterface</hardwareInterface>
+                    <hardwareInterface>hardware_interface/EffortJointInterface</hardwareInterface>
             </joint>
             <actuator name="z_back_wheel_motor">
-                    <hardwareInterface>EffortJointInterface</hardwareInterface>
+                    <hardwareInterface>hardware_interface/EffortJointInterface</hardwareInterface>
                     <mechanicalReduction>1</mechanicalReduction>
             </actuator>
@@ -35,8 +35,8 @@
             <type>transmission_interface/SimpleTransmission</type>
             <joint name="z_front_wheel_joint">
-                    <hardwareInterface>EffortJointInterface</hardwareInterface>
+                    <hardwareInterface>hardware_interface/EffortJointInterface</hardwareInterface>
             </joint>
             <actuator name="z_front_wheel_motor">
-                    <hardwareInterface>EffortJointInterface</hardwareInterface>
+                    <hardwareInterface>hardware_interface/EffortJointInterface</hardwareInterface>
                     <mechanicalReduction>1</mechanicalReduction>
             </actuator>

File: urdfs/flywheel.xacro (robot description, xacro)
@@ -5,5 +5,5 @@
     <xacro:include filename="$(find solo_description)/urdfs/flywheel.transmission.xacro"/>
     <xacro:include filename="$(find solo_description)/urdfs/flywheel.gazebo.xacro"/>
-    <joint name="z_left_wheel_joint" type="continuous">
+    <joint name="z_left_wheel_joint" type="revolute">
     <parent link="trunk"/>
     <child link="left_wheel"/>
@@ -11,9 +11,10 @@
     <axis xyz="0 0 1"/>
     <dynamics damping="0.1" friction="0.0"/>
+    <limit effort="1000" lower="-1e06" upper="1e06" velocity="1000"/>
     </joint>
     <link name="left_wheel">
     <inertial>
     <mass value="${mass_lr}"/>
-    <inertia ixx="0.001" ixy="0" ixz="0" iyy="0.001" iyz="0" izz="${inertia_lr}"/>
+    <inertia ixx="0.000001" ixy="0" ixz="0" iyy="0.000001" iyz="0" izz="${inertia_lr}"/>
     </inertial>
     <visual>
@@ -29,5 +30,5 @@
     </geometry>
     </collision>    </link>
-    <joint name="z_right_wheel_joint" type="continuous">
+    <joint name="z_right_wheel_joint" type="revolute">
     <parent link="trunk"/>
     <child link="right_wheel"/>
@@ -35,9 +36,10 @@
     <axis xyz="0 0 1"/>
     <dynamics damping="0.1" friction="0.0"/>
+    <limit effort="1000" lower="-1e06" upper="1e06" velocity="1000"/>
     </joint>
     <link name="right_wheel">
     <inertial>
     <mass value="${mass_lr}"/>
-    <inertia ixx="0.001" ixy="0" ixz="0" iyy="0.001" iyz="0" izz="${inertia_lr}"/>
+    <inertia ixx="0.000001" ixy="0" ixz="0" iyy="0.000001" iyz="0" izz="${inertia_lr}"/>
     </inertial>
     <visual>
@@ -54,5 +56,5 @@
     </collision>
     </link>
-    <joint name="z_front_wheel_joint" type="continuous">
+    <joint name="z_front_wheel_joint" type="revolute">
     <parent link="trunk"/>
     <child link="front_wheel"/>
@@ -60,9 +62,10 @@
     <axis xyz="0 0 1"/>
     <dynamics damping="0.1" friction="0.0"/>
+    <limit effort="1000" lower="-1e06" upper="1e06" velocity="1000"/>
     </joint>
     <link name="front_wheel">
     <inertial>
     <mass value="${mass_fh}"/>
-    <inertia ixx="0.001" ixy="0" ixz="0" iyy="0.001" iyz="0" izz="${inertia_fh}"/>
+    <inertia ixx="0.000001" ixy="0" ixz="0" iyy="0.000001" iyz="0" izz="${inertia_fh}"/>
     </inertial>
     <visual>
@@ -79,5 +82,5 @@
     </collision>
     </link>
-    <joint name="z_back_wheel_joint" type="continuous">
+    <joint name="z_back_wheel_joint" type="revolute">
     <parent link="trunk"/>
     <child link="back_wheel"/>
@@ -85,21 +88,22 @@
     <axis xyz="0 0 1"/>
     <dynamics damping="0.1" friction="0.0"/>
+    <limit effort="1000" lower="-1e06" upper="1e06" velocity="1000"/>
     </joint>
     <link name="back_wheel">
         <inertial>
-        <mass value="${mass_fh}"/>
-        <inertia ixx="0.001" ixy="0" ixz="0" iyy="0.001" iyz="0" izz="${inertia_fh}"/>
+            <mass value="${mass_fh}"/>
+            <inertia ixx="0.000001" ixy="0" ixz="0" iyy="0.000001" iyz="0" izz="${inertia_fh}"/>
         </inertial>
         <visual>
-        <origin rpy="0 0 0" xyz="0 0 0.0"/>
-        <geometry>
-        <cylinder length="0.05" radius="${radius}"/>
-        </geometry>
+            <origin rpy="0 0 0" xyz="0 0 0.0"/>
+            <geometry>
+            <cylinder length="0.05" radius="${radius}"/>
+            </geometry>
         </visual>
         <collision>
-        <origin rpy="0 0 0" xyz="0 0 0.0"/>
-        <geometry>
-        <cylinder length="0.05" radius="${radius}"/>
-        </geometry>
+            <origin rpy="0 0 0" xyz="0 0 0.0"/>
+            <geometry>
+            <cylinder length="0.05" radius="${radius}"/>
+            </geometry>
         </collision>
     </link>

Commit message: added compatibility with gazebo 11

File: robots/solo.urdf.xacro (robot description, xacro)
@@ -6,20 +6,23 @@
   <xacro:arg name="flywheel" default="false"/>
   <xacro:arg name="load_force_sensors" default="false"/>
+  <xacro:arg name="new_gazebo_version" default="false"/>
         <xacro:include filename="$(find solo_description)/gazebo/gazebo.urdf.xacro">
              <xacro:arg name="task_period" value="$(arg task_period)"/>
         </xacro:include>
-                <!-- Floating-base Joint -->
-                <link name="world"/>
-                <joint name="floating_base_joint" type="floating">
-                    <origin rpy="0 0 0" xyz="0 0 0"/>
-                    <parent link="world"/>
-                    <child link="base_link"/>
-                </joint>
-		<link name="base_link" />
-                <joint name="floating_base" type="fixed">
-                    <origin rpy="0 0 0" xyz="0 0 0"/>
-                    <parent link="base_link"/>
-                    <child link="trunk"/>
-                </joint>
+	   <xacro:unless value="$(arg new_gazebo_version)">
+		        <!-- Floating-base Joint -->
+		        <link name="world"/>
+		        <joint name="floating_base_joint" type="floating">
+		            <origin rpy="0 0 0" xyz="0 0 0"/>
+		            <parent link="world"/>
+		            <child link="base_link"/>
+		        </joint>
+			<link name="base_link" />
+		        <joint name="floating_base" type="fixed">
+		            <origin rpy="0 0 0" xyz="0 0 0"/>
+		            <parent link="base_link"/>
+		            <child link="trunk"/>
+		        </joint>
+	     </xacro:unless>
 		<link name="trunk">
 			<inertial>

Commit message: bugfix in floating joint

File: robots/solo.urdf.xacro (robot description, xacro)
@@ -10,19 +10,19 @@
              <xacro:arg name="task_period" value="$(arg task_period)"/>
         </xacro:include>
-	   <xacro:unless value="$(arg new_gazebo_version)">
+	     <xacro:unless value="$(arg new_gazebo_version)">
 		        <!-- Floating-base Joint -->
 		        <link name="world"/>
-		        <joint name="floating_base_joint" type="floating">
+		        <joint name="floating_base_joint" type="floating" >
 		            <origin rpy="0 0 0" xyz="0 0 0"/>
 		            <parent link="world"/>
 		            <child link="base_link"/>
 		        </joint>
-			<link name="base_link" />
+	     </xacro:unless>
+	     	<link name="base_link" />
 		        <joint name="floating_base" type="fixed">
 		            <origin rpy="0 0 0" xyz="0 0 0"/>
 		            <parent link="base_link"/>
 		            <child link="trunk"/>
-		        </joint>
-	     </xacro:unless>
+		</joint>
 		<link name="trunk">
 			<inertial>

Commit message: better tuned inertia and removed damping from flywheel

File: robots/solo.urdf.xacro (robot description, xacro)
@@ -63,6 +63,6 @@
         <xacro:if value="$(arg flywheel)">
               <xacro:include filename="$(find solo_description)/urdfs/flywheel.xacro"/>
-              <!-- inertia = 0.5 m*radius^2 but I had to set 10 times more for sm stability-->
-              <xacro:flywheel_train radius="0.05" mass_lr="0.2" inertia_lr="0.0025"  mass_fh="0.2" inertia_fh="0.0025"/>
+              <!-- inertia =  m*radius^2 but I had to set 10 times more for sm stability-->
+              <xacro:flywheel_train radius="0.05" mass_lr="0.1" inertia_lr="0.00025"  mass_fh="0.1" inertia_fh="0.00025"/>
         </xacro:if>
   <!-- Include the front left leg -->

File: urdfs/flywheel.xacro (robot description, xacro)
@@ -10,5 +10,5 @@
     <origin rpy="-1.57 0 0" xyz=" 0 0.15 0.0"/>
     <axis xyz="0 0 1"/>
-    <dynamics damping="0.1" friction="0.0"/>
+    <dynamics damping="0.0" friction="0.0"/>
     <limit effort="1000" lower="-1e06" upper="1e06" velocity="1000"/>
     </joint>
@@ -35,5 +35,5 @@
     <origin rpy="1.57 0 0" xyz=" 0 -0.15 0.0"/>
     <axis xyz="0 0 1"/>
-    <dynamics damping="0.1" friction="0.0"/>
+    <dynamics damping="0.0" friction="0.0"/>
     <limit effort="1000" lower="-1e06" upper="1e06" velocity="1000"/>
     </joint>
@@ -61,5 +61,5 @@
     <origin rpy="0.0 1.57 0" xyz=" 0.2 0.0 0.0"/>
     <axis xyz="0 0 1"/>
-    <dynamics damping="0.1" friction="0.0"/>
+    <dynamics damping="0.0" friction="0.0"/>
     <limit effort="1000" lower="-1e06" upper="1e06" velocity="1000"/>
     </joint>
@@ -87,5 +87,5 @@
     <origin rpy="0 -1.57 0" xyz=" -0.2 0.0 0.0"/>
     <axis xyz="0 0 1"/>
-    <dynamics damping="0.1" friction="0.0"/>
+    <dynamics damping="0.0" friction="0.0"/>
     <limit effort="1000" lower="-1e06" upper="1e06" velocity="1000"/>
     </joint>

Commit message: typo correction

File: robots/solo.urdf.xacro (robot description, xacro)
@@ -6,7 +6,7 @@
     <xacro:arg name="flywheel" default="false"/>
     <xacro:arg name="load_force_sensors" default="false"/>
-    <xacro:arg name="new_gazebo_version" default="true"/>
+    <xacro:arg name="new_gazebo_version" default="false"/>
     <xacro:include filename="$(find solo_description)/gazebo/gazebo.urdf.xacro">
-         <xacro:arg name="task_period" value="$(arg task_period)"/>
+        <xacro:arg name="task_period" value="$(arg task_period)"/>
     </xacro:include>
     <!-- BASE LINK -->
@@ -32,7 +32,7 @@
             <mass value="1.16115091"/>
             <!-- The base is extremely symmetrical. -->
-            <inertia ixx="0.00578574" ixy="0.0"        ixz="0.0"
-                                      iyy="0.01938108" iyz="0.0"
-                                                       izz="0.02476124"/>
+            <inertia ixx="0.00578574"   ixy="0.0"           ixz="0.0"
+                                        iyy="0.01938108"    iyz="0.0"
+                                                            izz="0.02476124"/>
         </inertial>
         <visual>
@@ -41,5 +41,5 @@
                 <mesh filename="package://solo_description/meshes/stl/with_foot/solo_body.stl"/>
             </geometry>
-            <material name="${color_name}">
+                <material name="${color_name}">
                 <color rgba="${color} ${opacity}"/>
             </material>
@@ -56,55 +56,55 @@
         <!-- Bullet specific paramters -->
         <contact>
-        <lateral_friction value="1.0"/>
-        <restitution value="0.5"/>
+            <lateral_friction value="1.0"/>
+            <restitution value="0.5"/>
         </contact>
     </link>
-    <!-- Include legs -->
+    <!-- Include the legs -->
     <xacro:include filename="$(find solo_description)/urdfs/leg.xacro"/>
     <!-- Include flywheels -->
     <xacro:if value="$(arg flywheel)">
-          <xacro:include filename="$(find solo_description)/urdfs/flywheel.xacro"/>
-          <!-- inertia =  m*radius^2 but I had to set 10 times more for sm stability-->
-          <xacro:flywheel_train radius="0.05" mass_lr="0.1" inertia_lr="0.00025"  mass_fh="0.1" inertia_fh="0.00025"/>
+        <xacro:include filename="$(find solo_description)/urdfs/flywheel.xacro"/>
+        <!-- inertia =  m*radius^2 but I had to set 10 times more for sm stability-->
+        <xacro:flywheel_train radius="0.05" mass_lr="0.1" inertia_lr="0.00025"  mass_fh="0.1" inertia_fh="0.00025"/>
     </xacro:if>
     <!-- LEFT FRONT LEG -->
     <xacro:leg
-        prefix="lf"
-        is_front="true"
-        is_right="false"
-        has_side_motion="true"
-        color_name="${color_name}"
-        color="${color}"
-        opacity="${opacity}"
-        load_force_sensors="$(arg load_force_sensors)"/>
+    prefix="lf"
+    is_front="true"
+    is_right="false"
+    has_side_motion="true"
+    color_name="${color_name}"
+    color="${color}"
+    opacity="${opacity}"
+    load_force_sensors="$(arg load_force_sensors)"/>
     <!-- RIGHT FRONT LEG -->
     <xacro:leg
-        prefix="rf"
-        is_front="true"
-        is_right="true"
-        has_side_motion="true"
-        color_name="${color_name}"
-        color="${color}"
-        opacity="${opacity}"
-        load_force_sensors="$(arg load_force_sensors)"/>
+    prefix="rf"
+    is_front="true"
+    is_right="true"
+    has_side_motion="true"
+    color_name="${color_name}"
+    color="${color}"
+    opacity="${opacity}"
+    load_force_sensors="$(arg load_force_sensors)"/>
     <!-- LEFT HIND LEG -->
     <xacro:leg
-        prefix="lh"
-        is_front="false"
-        is_right="false"
-        has_side_motion="true"
-        color_name="${color_name}"
-        color="${color}"
-        opacity="${opacity}"
-        load_force_sensors="$(arg load_force_sensors)"/>
+    prefix="lh"
+    is_front="false"
+    is_right="false"
+    has_side_motion="true"
+    color_name="${color_name}"
+    color="${color}"
+    opacity="${opacity}"
+    load_force_sensors="$(arg load_force_sensors)"/>
     <!-- RIGHT HIND LEG -->
     <xacro:leg
-        prefix="rh"
-        is_front="false"
-        is_right="true"
-        has_side_motion="true"
-        color_name="${color_name}"
-        color="${color}"
-        opacity="${opacity}"
-        load_force_sensors="$(arg load_force_sensors)"/>
+    prefix="rh"
+    is_front="false"
+    is_right="true"
+    has_side_motion="true"
+    color_name="${color_name}"
+    color="${color}"
+    opacity="${opacity}"
+    load_force_sensors="$(arg load_force_sensors)"/>
 </robot>
