Commit message: bug fix: correct files for mash are loaded now

File: robots/solo.urdf.xacro (robot description, xacro)
@@ -39,5 +39,6 @@
             <origin xyz="0 0 0" rpy="0 0 0" />
             <geometry>
-                <mesh filename="package://solo_description/meshes/stl/with_foot/solo_body.stl"/>
+                <!-- mesh filename="package://solo_description/meshes/stl/with_foot/solo_body.stl"/ -->
+                <mesh filename="package://solo_description/meshes/stl/solo12/solo12_base.stl"/>
             </geometry>
                 <material name="${color_name}">
@@ -48,5 +49,6 @@
             <origin xyz="0 0 0" rpy="0 0 0" />
             <geometry>
-                <mesh filename="package://solo_description/meshes/stl/with_foot/solo_body.stl"/>
+                <!-- mesh filename="package://solo_description/meshes/stl/with_foot/solo_body.stl"/ -->
+                <mesh filename="package://solo_description/meshes/stl/solo12/solo12_base.stl"/>
             </geometry>
             <material name="${color_name}">

File: urdfs/leg.xacro (robot description, xacro)
@@ -14,5 +14,5 @@
     <xacro:property name="KFE_2_FOOT_y" value="${8.0 * 0.001}" />
     <xacro:property name="KFE_2_FOOT_z" value="${160.00 * 0.001}" />
-    <xacro:property name="MAX_TORQUE" value="1.2" />
+    <xacro:property name="MAX_TORQUE" value="1.7" />
     <!-- This macro has for purpose to define a leg -->
     <xacro:macro name="leg" params="prefix is_front is_right has_side_motion
@@ -271,8 +271,10 @@
                 <geometry>
                     <xacro:unless value="${is_right}">
-                        <mesh filename="package://solo_description/meshes/stl/with_foot/solo_upper_leg_left_side.stl"/>
-                    </xacro:unless>
-                    <xacro:if value="${is_right}">
-                        <mesh filename="package://solo_description/meshes/stl/with_foot/solo_upper_leg_right_side.stl"/>
+                        <!--mesh filename="package://solo_description/meshes/stl/with_foot/solo_upper_leg_left_side.stl"/-->
+                        <mesh filename="package://solo_description/meshes/stl/solo12/solo12_upper_leg_left_side.stl"/>
+                    </xacro:unless>
+                    <xacro:if value="${is_right}">
+                        <!--mesh filename="package://solo_description/meshes/stl/with_foot/solo_upper_leg_right_side.stl"/-->
+                        <mesh filename="package://solo_description/meshes/stl/solo12/solo12_upper_leg_right_side.stl"/>
                     </xacro:if>
                 </geometry>
@@ -286,8 +288,10 @@
                 <geometry>
                     <xacro:unless value="${is_right}">
-                        <mesh filename="package://solo_description/meshes/stl/with_foot/solo_upper_leg_left_side.stl"/>
-                    </xacro:unless>
-                    <xacro:if value="${is_right}">
-                        <mesh filename="package://solo_description/meshes/stl/with_foot/solo_upper_leg_right_side.stl"/>
+                        <!--mesh filename="package://solo_description/meshes/stl/with_foot/solo_upper_leg_left_side.stl"/-->
+                        <mesh filename="package://solo_description/meshes/stl/solo12/solo12_upper_leg_left_side.stl"/>
+                    </xacro:unless>
+                    <xacro:if value="${is_right}">
+                        <!--mesh filename="package://solo_description/meshes/stl/with_foot/solo_upper_leg_right_side.stl"/-->
+                        <mesh filename="package://solo_description/meshes/stl/solo12/solo12_upper_leg_right_side.stl"/>
                     </xacro:if>
                 </geometry>
@@ -368,8 +372,10 @@
                 <geometry>
                     <xacro:unless value="${is_right}">
-                        <mesh filename="package://solo_description/meshes/stl/with_foot/solo_lower_leg_left_side.stl"/>
-                    </xacro:unless>
-                    <xacro:if value="${is_right}">
-                        <mesh filename="package://solo_description/meshes/stl/with_foot/solo_lower_leg_right_side.stl"/>
+                        <!--mesh filename="package://solo_description/meshes/stl/with_foot/solo_lower_leg_left_side.stl"/-->
+                        <mesh filename="package://solo_description/meshes/stl/solo12/solo12_lower_leg_left_side.stl"/>
+                    </xacro:unless>
+                    <xacro:if value="${is_right}">
+                        <!--mesh filename="package://solo_description/meshes/stl/with_foot/solo_lower_leg_right_side.stl"/-->
+                        <mesh filename="package://solo_description/meshes/stl/solo12/solo12_lower_leg_right_side.stl"/>
                     </xacro:if>
                 </geometry>
@@ -383,8 +389,10 @@
                 <geometry>
                     <xacro:unless value="${is_right}">
-                        <mesh filename="package://solo_description/meshes/stl/with_foot/solo_lower_leg_left_side.stl"/>
-                    </xacro:unless>
-                    <xacro:if value="${is_right}">
-                        <mesh filename="package://solo_description/meshes/stl/with_foot/solo_lower_leg_right_side.stl"/>
+                        <!--mesh filename="package://solo_description/meshes/stl/with_foot/solo_lower_leg_left_side.stl"/-->
+                        <mesh filename="package://solo_description/meshes/stl/solo12/solo12_lower_leg_left_side.stl"/>
+                    </xacro:unless>
+                    <xacro:if value="${is_right}">
+                        <!--mesh filename="package://solo_description/meshes/stl/with_foot/solo_lower_leg_right_side.stl"/-->
+                        <mesh filename="package://solo_description/meshes/stl/solo12/solo12_lower_leg_right_side.stl"/>
                     </xacro:if>
                 </geometry>
@@ -428,4 +436,5 @@
                 <origin xyz="0 0 0" rpy="0 0 0" />
                 <geometry>
+                    <!-- mesh filename="package://solo_description/meshes/stl/with_foot/solo_foot.stl"/ -->
                     <mesh filename="package://solo_description/meshes/stl/with_foot/solo_foot.stl"/>
                 </geometry>
@@ -438,6 +447,7 @@
                 <origin xyz="0 0 0" rpy="0 0 0" />
                 <geometry>
-                    <mesh filename="package://solo_description/meshes/stl/with_foot/solo_foot.stl"/>
-                    <!-- sphere radius="0.01"/-->
+                    <!-- mesh filename="package://solo_description/meshes/stl/with_foot/solo_foot.stl"/ -->
+                    <mesh filename="package://solo_description/meshes/stl/with_foot/solo_foot.stl"/>>
+                    <!--sphere radius="0.01"/-->
                 </geometry>
                 <material name="${color_name}">
@@ -447,8 +457,9 @@
             <!-- Bullet specific paramters -->
             <contact>
-                <lateral_friction value="1.0"/>
-                <restitution value="0.5"/>
+                <lateral_friction value="0.8"/>
+                <restitution value="0.0"/>
             </contact>
-        </link> <!-- END FOOT LINK -->
+        </link>
+        <!-- END FOOT LINK -->
         <!-- Extensions -->
         <xacro:leg_transmission name="${prefix}"/>

Commit message: bug fix: correct files for mash are loaded now

File: robots/solo.urdf.xacro (robot description, xacro)
@@ -39,6 +39,5 @@
             <origin xyz="0 0 0" rpy="0 0 0" />
             <geometry>
-                <!-- mesh filename="package://solo_description/meshes/stl/with_foot/solo_body.stl"/ -->
-                <mesh filename="package://solo_description/meshes/stl/solo12/solo12_base.stl"/>
+                <mesh filename="package://solo_description/meshes/stl/with_foot/solo_body.stl"/>
             </geometry>
                 <material name="${color_name}">
@@ -49,6 +48,5 @@
             <origin xyz="0 0 0" rpy="0 0 0" />
             <geometry>
-                <!-- mesh filename="package://solo_description/meshes/stl/with_foot/solo_body.stl"/ -->
-                <mesh filename="package://solo_description/meshes/stl/solo12/solo12_base.stl"/>
+                <mesh filename="package://solo_description/meshes/stl/with_foot/solo_body.stl"/>
             </geometry>
             <material name="${color_name}">

File: urdfs/leg.xacro (robot description, xacro)
@@ -14,5 +14,5 @@
     <xacro:property name="KFE_2_FOOT_y" value="${8.0 * 0.001}" />
     <xacro:property name="KFE_2_FOOT_z" value="${160.00 * 0.001}" />
-    <xacro:property name="MAX_TORQUE" value="1.7" />
+    <xacro:property name="MAX_TORQUE" value="1.2" />
     <!-- This macro has for purpose to define a leg -->
     <xacro:macro name="leg" params="prefix is_front is_right has_side_motion
@@ -271,10 +271,8 @@
                 <geometry>
                     <xacro:unless value="${is_right}">
-                        <!--mesh filename="package://solo_description/meshes/stl/with_foot/solo_upper_leg_left_side.stl"/-->
-                        <mesh filename="package://solo_description/meshes/stl/solo12/solo12_upper_leg_left_side.stl"/>
-                    </xacro:unless>
-                    <xacro:if value="${is_right}">
-                        <!--mesh filename="package://solo_description/meshes/stl/with_foot/solo_upper_leg_right_side.stl"/-->
-                        <mesh filename="package://solo_description/meshes/stl/solo12/solo12_upper_leg_right_side.stl"/>
+                        <mesh filename="package://solo_description/meshes/stl/with_foot/solo_upper_leg_left_side.stl"/>
+                    </xacro:unless>
+                    <xacro:if value="${is_right}">
+                        <mesh filename="package://solo_description/meshes/stl/with_foot/solo_upper_leg_right_side.stl"/>
                     </xacro:if>
                 </geometry>
@@ -288,10 +286,8 @@
                 <geometry>
                     <xacro:unless value="${is_right}">
-                        <!--mesh filename="package://solo_description/meshes/stl/with_foot/solo_upper_leg_left_side.stl"/-->
-                        <mesh filename="package://solo_description/meshes/stl/solo12/solo12_upper_leg_left_side.stl"/>
-                    </xacro:unless>
-                    <xacro:if value="${is_right}">
-                        <!--mesh filename="package://solo_description/meshes/stl/with_foot/solo_upper_leg_right_side.stl"/-->
-                        <mesh filename="package://solo_description/meshes/stl/solo12/solo12_upper_leg_right_side.stl"/>
+                        <mesh filename="package://solo_description/meshes/stl/with_foot/solo_upper_leg_left_side.stl"/>
+                    </xacro:unless>
+                    <xacro:if value="${is_right}">
+                        <mesh filename="package://solo_description/meshes/stl/with_foot/solo_upper_leg_right_side.stl"/>
                     </xacro:if>
                 </geometry>
@@ -372,10 +368,8 @@
                 <geometry>
                     <xacro:unless value="${is_right}">
-                        <!--mesh filename="package://solo_description/meshes/stl/with_foot/solo_lower_leg_left_side.stl"/-->
-                        <mesh filename="package://solo_description/meshes/stl/solo12/solo12_lower_leg_left_side.stl"/>
-                    </xacro:unless>
-                    <xacro:if value="${is_right}">
-                        <!--mesh filename="package://solo_description/meshes/stl/with_foot/solo_lower_leg_right_side.stl"/-->
-                        <mesh filename="package://solo_description/meshes/stl/solo12/solo12_lower_leg_right_side.stl"/>
+                        <mesh filename="package://solo_description/meshes/stl/with_foot/solo_lower_leg_left_side.stl"/>
+                    </xacro:unless>
+                    <xacro:if value="${is_right}">
+                        <mesh filename="package://solo_description/meshes/stl/with_foot/solo_lower_leg_right_side.stl"/>
                     </xacro:if>
                 </geometry>
@@ -389,10 +383,8 @@
                 <geometry>
                     <xacro:unless value="${is_right}">
-                        <!--mesh filename="package://solo_description/meshes/stl/with_foot/solo_lower_leg_left_side.stl"/-->
-                        <mesh filename="package://solo_description/meshes/stl/solo12/solo12_lower_leg_left_side.stl"/>
-                    </xacro:unless>
-                    <xacro:if value="${is_right}">
-                        <!--mesh filename="package://solo_description/meshes/stl/with_foot/solo_lower_leg_right_side.stl"/-->
-                        <mesh filename="package://solo_description/meshes/stl/solo12/solo12_lower_leg_right_side.stl"/>
+                        <mesh filename="package://solo_description/meshes/stl/with_foot/solo_lower_leg_left_side.stl"/>
+                    </xacro:unless>
+                    <xacro:if value="${is_right}">
+                        <mesh filename="package://solo_description/meshes/stl/with_foot/solo_lower_leg_right_side.stl"/>
                     </xacro:if>
                 </geometry>
@@ -436,5 +428,4 @@
                 <origin xyz="0 0 0" rpy="0 0 0" />
                 <geometry>
-                    <!-- mesh filename="package://solo_description/meshes/stl/with_foot/solo_foot.stl"/ -->
                     <mesh filename="package://solo_description/meshes/stl/with_foot/solo_foot.stl"/>
                 </geometry>
@@ -447,7 +438,6 @@
                 <origin xyz="0 0 0" rpy="0 0 0" />
                 <geometry>
-                    <!-- mesh filename="package://solo_description/meshes/stl/with_foot/solo_foot.stl"/ -->
-                    <mesh filename="package://solo_description/meshes/stl/with_foot/solo_foot.stl"/>>
-                    <!--sphere radius="0.01"/-->
+                    <mesh filename="package://solo_description/meshes/stl/with_foot/solo_foot.stl"/>
+                    <!-- sphere radius="0.01"/-->
                 </geometry>
                 <material name="${color_name}">
@@ -457,9 +447,8 @@
             <!-- Bullet specific paramters -->
             <contact>
-                <lateral_friction value="0.8"/>
-                <restitution value="0.0"/>
+                <lateral_friction value="1.0"/>
+                <restitution value="0.5"/>
             </contact>
-        </link>
-        <!-- END FOOT LINK -->
+        </link> <!-- END FOOT LINK -->
         <!-- Extensions -->
         <xacro:leg_transmission name="${prefix}"/>

Commit message: introduced PI and angle->angle_deg

File: robots/solo.urdf.xacro (robot description, xacro)
@@ -6,5 +6,5 @@
     <xacro:arg name="flywheel" default="false"/>
     <xacro:arg name="flywheel2" default="true"/>
-    <xacro:arg name="angle" default="0.0"/>
+    <xacro:arg name="angle_deg" default="0.0"/>
     <xacro:arg name="load_force_sensors" default="false"/>
     <xacro:arg name="new_gazebo_version" default="false"/>
@@ -74,5 +74,5 @@
         <xacro:include filename="$(find solo_description)/urdfs/flywheel2.xacro"/>
         <!-- inertia =  m*radius^2 but I had to set 10 times more for sm stability-->
-        <xacro:flywheel_train radius="0.03" height="0.01" mass="0.1" inertia_z="0.000068" inertia_xy="0.000037" angle="$(arg angle)"/>
+        <xacro:flywheel_train radius="0.03" height="0.01" mass="0.1" inertia_z="0.000068" inertia_xy="0.000037" angle_deg="$(arg angle_deg)"/>
     </xacro:if>
     <!-- LEFT FRONT LEG -->

File: urdfs/flywheel2.xacro (robot description, xacro)
@@ -2,11 +2,13 @@
 <robot xmlns:xacro="http://ros.org/wiki/xacro" name="solo">
     <!-- Things that are needed only for Gazebo (not the physical robot). These include sensor and controller plugin specifications -->
-    <xacro:macro name="flywheel_train" params="radius height mass inertia_z inertia_xy angle">
+    <xacro:macro name="flywheel_train" params="radius height mass inertia_z inertia_xy angle_deg">
         <xacro:include filename="$(find solo_description)/urdfs/flywheel2.transmission.xacro"/>
         <xacro:include filename="$(find solo_description)/urdfs/flywheel2.gazebo.xacro"/>
+        <xacro:property name="PI" value="3.1415926535897931"/>
+        <xacro:property name="angle_rad" value="${angle_deg * PI / 180}"/>
         <joint name="z_left_wheel_joint" type="revolute">
             <parent link="trunk"/>
             <child link="left_wheel"/>
-            <origin rpy="-1.57 0 -${angle}" xyz="${-0.025 +0.025*cos(angle) +0.02*sin(angle)} ${+0.047 -0.025*sin(angle) +0.02*cos(angle)} 0.066"/>
+            <origin rpy="${-PI/2} 0 -${angle_rad}" xyz="${-0.025 +0.025*cos(angle_rad) +0.02*sin(angle_rad)} ${+0.047 -0.025*sin(angle_rad) +0.02*cos(angle_rad)} 0.066"/>
             <axis xyz="0 0 1"/>
             <dynamics damping="0.0" friction="0.0"/>
@@ -24,5 +26,5 @@
                 <origin rpy="0 0 0" xyz="0 0 0.0"/>
                 <geometry>
-                    <mesh scale="0.001 0.001 0.001" filename="package://solo_description/meshes/stl/flywheel/flywheel.stl"/>
+                    <mesh scale="0.001 0.001 0.001" filename="package://solo_description/meshes/stl/flywheel/flywheel.stl"/> <!--the measure in the stl files are expressed in mm-->
                 </geometry>
             </visual>
@@ -37,5 +39,5 @@
             <parent link="trunk"/>
             <child link="right_wheel"/>
-            <origin rpy="1.57 0 ${angle}" xyz="${-0.025 +0.025*cos(angle)+0.02*sin(angle)} ${-0.047 +0.025*sin(angle) -0.02*cos(angle)} 0.066"/>
+            <origin rpy="${PI/2} 0 ${angle_rad}" xyz="${-0.025 +0.025*cos(angle_rad)+0.02*sin(angle_rad)} ${-0.047 +0.025*sin(angle_rad) -0.02*cos(angle_rad)} 0.066"/>
             <axis xyz="0 0 1"/>
             <dynamics damping="0.0" friction="0.0"/>

Commit message: finally fixing the hack of new_gazebo_version to set root joint for pinocchio as per robot_control commit fccb58b1fb819f6c18701ba5d1a20bd6d21af330

File: robots/solo.urdf.xacro (robot description, xacro)
@@ -7,20 +7,8 @@
     <xacro:arg name="robot_name" default="solo"/>
     <xacro:arg name="angle_deg" default="0.0"/>
-    <xacro:arg name="new_gazebo_version" default="false"/>
     <xacro:include filename="$(find solo_description)/gazebo/gazebo.urdf.xacro">
         <xacro:arg name="task_period" value="$(arg task_period)"/>
 	<xacro:arg name="robot_name" value="$(arg robot_name)"/>
     </xacro:include>
-    <!-- BASE LINK -->
-    <!-- floating type is supported in older versions of Gazebo. In new Gazebo if a link has no parent, it is supposed to be attached to a floating joint -->
-    <xacro:unless value="$(arg new_gazebo_version)">
-        <!-- Floating-base Joint -->
-        <link name="world"/>
-        <joint name="floating_base_joint" type="floating" >
-            <origin rpy="0 0 0" xyz="0 0 0"/>
-            <parent link="world"/>
-            <child link="base_link"/>
-        </joint>
-    </xacro:unless>
     <link name="base_link" />
     <joint name="floating_base" type="fixed">
