Commit message: cleaned up stuff and now working with rviz (still feet are out)

File: gazebo/gazebo.urdf.xacro (robot description, xacro)
@@ -4,10 +4,11 @@
 	<gazebo>
 		<plugin name="gazebo_ros_controller_manager" filename="libgazebo_ros_control.so">
-                        <robotNamespace>/solo</robotNamespace>
-                        <robotSimType>dls_gazebo_interface/DlsRobotHwSim</robotSimType>
-                        <controlPeriod>$(arg task_period)</controlPeriod>
+			<robotNamespace>/solo12</robotNamespace>
+			<robotSimType>gazebo_ros_control/DefaultRobotHWSim</robotSimType>
+			<legacyModeNS>true</legacyModeNS>
+            		<controlPeriod>$(arg task_period)</controlPeriod>
 		</plugin>
 		<plugin filename="libgazebo_ros_p3d.so" name="gazebo_ros_p3d">
-                        <robotNamespace>/solo</robotNamespace>
+                        <robotNamespace>/solo12</robotNamespace>
                         <bodyName>trunk</bodyName>
 			<topicName>ground_truth</topicName>

File: urdfs/leg.gazebo.xacro (robot description, xacro)
@@ -8,5 +8,5 @@
                         <gazebo>
                                 <plugin name="${name}_haa_sensor" filename="libgazebo_ros_ft_sensor.so">
-                                        <robotNamespace>/solo/internal_wrench/</robotNamespace>
+                                        <robotNamespace>/solo12/internal_wrench/</robotNamespace>
                                         <updateRate>100.0</updateRate>
                                         <topicName>${name}_haa_joint</topicName>
@@ -21,5 +21,5 @@
                         <gazebo>
                                 <plugin name="${name}_kfe_sensor" filename="libgazebo_ros_ft_sensor.so">
-                                        <robotNamespace>/solo/internal_wrench/</robotNamespace>
+                                        <robotNamespace>/solo12/internal_wrench/</robotNamespace>
                                         <updateRate>100.0</updateRate>
                                         <topicName>${name}_kfe_joint</topicName>
@@ -34,5 +34,5 @@
                         <gazebo>
                                 <plugin name="${name}_hfe_sensor" filename="libgazebo_ros_ft_sensor.so">
-                                        <robotNamespace>/solo/internal_wrench/</robotNamespace>
+                                        <robotNamespace>/solo12/internal_wrench/</robotNamespace>
                                         <updateRate>100.0</updateRate>
                                         <topicName>${name}_hfe_joint</topicName>
@@ -66,5 +66,5 @@
                 because gazebo lumps the fake footframe with the real parent link, the normals are in the world frame-->
                  <plugin name="${name}_shin_bumper" filename="libgazebo_ros_bumper.so">
-                  <bumperTopicName>/solo/${name}_shin_bumper</bumperTopicName>
+                  <bumperTopicName>/solo12/${name}_shin_bumper</bumperTopicName>
                 </plugin>
             </sensor>
@@ -86,6 +86,6 @@
                                 because gazebo lumps the fake footframe with the real parent link, the normals are in the world frame-->
                                 <plugin name="${name}_foot_bumper" filename="libgazebo_ros_bumper.so">
-                                        <bumperTopicName>/solo/${name}_foot_bumper</bumperTopicName>
-                                        <robotNamespace>solo</robotNamespace>
+                                        <bumperTopicName>/solo12/${name}_foot_bumper</bumperTopicName>
+                                        <robotNamespace>solo12</robotNamespace>
                                 </plugin>
                         </sensor>

File: urdfs/leg.transmission.xacro (robot description, xacro)
@@ -6,8 +6,8 @@
                         <type>transmission_interface/SimpleTransmission</type>
                         <joint name="${name}_haa_joint">
-                                <hardwareInterface>EffortJointInterface</hardwareInterface>
+                                <hardwareInterface>hardware_interface/EffortJointInterface</hardwareInterface>
                         </joint>
                         <actuator name="${name}_haa_motor">
-                                <hardwareInterface>EffortJointInterface</hardwareInterface>
+                                <hardwareInterface>hardware_interface/EffortJointInterface</hardwareInterface>
                                 <mechanicalReduction>1</mechanicalReduction>
                         </actuator>
@@ -17,8 +17,8 @@
                         <type>transmission_interface/SimpleTransmission</type>
                         <joint name="${name}_hfe_joint">
-                                <hardwareInterface>EffortJointInterface</hardwareInterface>
+                                <hardwareInterface>hardware_interface/EffortJointInterface</hardwareInterface>
                         </joint>
                         <actuator name="${name}_hfe_motor">
-                                <hardwareInterface>EffortJointInterface</hardwareInterface>
+                                <hardwareInterface>hardware_interface/EffortJointInterface</hardwareInterface>
                                 <mechanicalReduction>1</mechanicalReduction>
                         </actuator>
@@ -28,8 +28,8 @@
                         <type>transmission_interface/SimpleTransmission</type>
                         <joint name="${name}_kfe_joint">
-                                <hardwareInterface>EffortJointInterface</hardwareInterface>
+                                <hardwareInterface>hardware_interface/EffortJointInterface</hardwareInterface>
                         </joint>
                         <actuator name="${name}_kfe_motor">
-                                <hardwareInterface>EffortJointInterface</hardwareInterface>
+                                <hardwareInterface>hardware_interface/EffortJointInterface</hardwareInterface>
                                 <mechanicalReduction>1</mechanicalReduction>
                         </actuator>

File: xacro/solo12.srdf.xacro (robot description, xacro)
@@ -1,4 +1,3 @@
-<?xml version="1.0" ?>
-<robot name="solo" xmlns:xacro="http://ros.org/wiki/xacro">
+<robot name="solo12" xmlns:xacro="http://ros.org/wiki/xacro">
   <group name="base">
     <link name="base_link"/>
@@ -23,16 +22,16 @@
   </group>
   <group_state group="chains" name="home">
-    <joint name="lf_haa_joint" value="0.0"/>
+    <joint name="lf_haa_joint" value="-0.2"/>
     <joint name="lf_hfe_joint" value="0.75"/>
-    <joint name="lf_kfe_joint" value="-1.0"/>
-    <joint name="rf_haa_joint" value="0.0"/>
+    <joint name="lf_kfe_joint" value="-1.5"/>
+    <joint name="rf_haa_joint" value="-0.2"/>
     <joint name="rf_hfe_joint" value="0.75"/>
-    <joint name="rf_kfe_joint" value="-1.0"/>
-    <joint name="lh_haa_joint" value="0.0"/>
-    <joint name="lh_hfe_joint" value="-0.75"/>
-    <joint name="lh_kfe_joint" value="1.0"/>
-    <joint name="rh_haa_joint" value="0.0"/>
-    <joint name="rh_hfe_joint" value="-0.75"/>
-    <joint name="rh_kfe_joint" value="1.0"/>
+    <joint name="rf_kfe_joint" value="-1.5"/>
+    <joint name="lh_haa_joint" value="-0.2"/>
+    <joint name="lh_hfe_joint" value="0.75"/>
+    <joint name="lh_kfe_joint" value="-1.5"/>
+    <joint name="rh_haa_joint" value="-0.2"/>
+    <joint name="rh_hfe_joint" value="0.75"/>
+    <joint name="rh_kfe_joint" value="-1.5"/>
   </group_state>
 </robot>

File: xacro/solo12.urdf.xacro (robot description, xacro)
@@ -1,4 +1,4 @@
 <?xml version="1.0" ?>
-<robot name="solo"
+<robot name="solo12"
   xmlns:controller="http://playerstage.sourceforge.net/gazebo/xmlschema/#controller"
   xmlns:interface="http://playerstage.sourceforge.net/gazebo/xmlschema/#interface"
@@ -9,67 +9,59 @@
   <xacro:property name="color" value="0.8 0.8 0.8" />
   <xacro:property name="opacity" value="1.0" />
-    <!-- Floating-base Joint -->
-    <link name="world"/>
-    <joint name="floating_base_joint" type="floating">
-        <origin rpy="0 0 0" xyz="0 0 0"/>
-        <parent link="world"/>
-        <child link="base_link"/>
-        </joint>
-        <joint name="floating_base" type="fixed">
-        <origin rpy="0 0 0" xyz="0 0 0"/>
-        <parent link="base_link"/>
-        <child link="trunk"/>
-    </joint>
-    <link name="trunk"/>
-    <!-- Fixed joint to add dummy inertia link -->
-    <joint name="base_to_base_inertia" type="fixed">
-        <parent link="trunk"/>
-        <child link="base_inertia"/>
-        <origin rpy="0 0 0" xyz="0 0 0"/>
-    </joint>
-    <!-- Dummy inertia link, because KDL cannot have inertia on the base link -->
-    <link name="base_inertia">
-        <inertial>
-            <origin xyz="0 0 0" rpy="0 0 0" />
-            <mass value="1.63315091"/>
-            <!-- The base is extremely symmetrical. -->
-            <inertia ixx="0.00578574" ixy="0.0" ixz="0.0"
-                                      iyy="0.01938108" iyz="0.0"
-                                                       izz="0.02476124"/>
-        </inertial>
-    </link>
-  <!-- This file is based on: https://atlas.is.localnet/confluence/display/AMDW/Quadruped+URDF+Files -->
-  <link name="base_link">
-                <!-- BASE LINK VISUAL -->
-                <visual>
-                    <origin xyz="0 0 0" rpy="0 0 0" />
-                    <geometry>
-                      <mesh filename="package://solo_description/meshes/stl/with_foot/solo_body.stl"/>
-                    </geometry>
-                    <material name="${color_name}">
-                        <color rgba="${color} ${opacity}"/>
-                    </material>
-                </visual>
-                <!-- BASE LINK COLLISION -->
-                <collision>
-                    <origin xyz="0 0 0" rpy="0 0 0" />
-                    <geometry>
-                      <mesh filename="package://solo_description/meshes/stl/with_foot/solo_body.stl"/>
-                    </geometry>
-                    <material name="${color_name}">
-                        <color rgba="${color} ${opacity}"/>
-                    </material>
-                </collision>
-                <!-- Bullet specific paramters -->
-                <contact>
-                  <lateral_friction value="1.0"/>
-                  <restitution value="0.5"/>
-                </contact>
-  </link> <!-- END BASE LINK -->
-  <!-- Include the legs -->
-  <xacro:include filename="leg.xacro"/>
+        <xacro:include filename="$(find solo_description)/gazebo/gazebo.urdf.xacro">
+             <xacro:arg name="task_period" value="$(arg task_period)"/>
+        </xacro:include>
+                <!-- Floating-base Joint -->
+                <link name="world"/>
+                <joint name="floating_base_joint" type="floating">
+                    <origin rpy="0 0 0" xyz="0 0 0"/>
+                    <parent link="world"/>
+                    <child link="base_link"/>
+                </joint>
+		<link name="base_link" />
+                <joint name="floating_base" type="fixed">
+                    <origin rpy="0 0 0" xyz="0 0 0"/>
+                    <parent link="base_link"/>
+                    <child link="trunk"/>
+                </joint>
+		<link name="trunk">
+			<inertial>
+			    <origin xyz="0 0 0" rpy="0 0 0" />
+			    <mass value="1.63315091"/>
+			    <!-- The base is extremely symmetrical. -->
+			    <inertia ixx="0.00578574" ixy="0.0" ixz="0.0"
+				                      iyy="0.01938108" iyz="0.0"
+				                                       izz="0.02476124"/>
+			</inertial>
+			<visual>
+				<origin xyz="0 0 0" rpy="0 0 0" />
+				    <geometry>
+				      <mesh filename="package://solo_description/meshes/stl/with_foot/solo_body.stl"/>
+				    </geometry>
+				    <material name="${color_name}">
+				        <color rgba="${color} ${opacity}"/>
+				    </material>
+			</visual>
+			<collision>
+		            <origin xyz="0 0 0" rpy="0 0 0" />
+		            <geometry>
+		              <mesh filename="package://solo_description/meshes/stl/with_foot/solo_body.stl"/>
+		            </geometry>
+		            <material name="${color_name}">
+		                <color rgba="${color} ${opacity}"/>
+		            </material>
+               		 </collision>
+			<!-- Bullet specific paramters -->
+		        <contact>
+		          <lateral_friction value="1.0"/>
+		          <restitution value="0.5"/>
+		        </contact>
+		</link>
+ 	 <!-- Include the legs -->
+  	<xacro:include filename="$(find solo_description)/urdfs/leg.xacro"/>
+	<xacro:arg name="task_period" default="0.004"/>
   <!-- Include the front left leg -->
   <xacro:leg
-      prefix="FL"
+      prefix="lf"
       is_front="true"
       is_right="false"
@@ -81,5 +73,5 @@
   <!-- Include the front right leg -->
   <xacro:leg
-      prefix="FR"
+      prefix="rf"
       is_front="true"
       is_right="true"
@@ -91,5 +83,5 @@
   <!-- Include the hind left leg -->
   <xacro:leg
-      prefix="HL"
+      prefix="lh"
       is_front="false"
       is_right="false"
@@ -101,5 +93,5 @@
   <!-- Include the hind right leg -->
   <xacro:leg
-      prefix="HR"
+      prefix="rh"
       is_front="false"
       is_right="true"

Commit message: renamed solo12 in solo
parametrized radius of flywheel

File: gazebo/gazebo.urdf.xacro (robot description, xacro)
@@ -4,5 +4,5 @@
 	<gazebo>
 		<plugin name="gazebo_ros_controller_manager" filename="libgazebo_ros_control.so">
-			<robotNamespace>/solo12</robotNamespace>
+			<robotNamespace>/solo</robotNamespace>
 			<robotSimType>gazebo_ros_control/DefaultRobotHWSim</robotSimType>
 			<legacyModeNS>true</legacyModeNS>
@@ -10,5 +10,5 @@
 		</plugin>
 		<plugin filename="libgazebo_ros_p3d.so" name="gazebo_ros_p3d">
-                        <robotNamespace>/solo12</robotNamespace>
+                        <robotNamespace>/solo</robotNamespace>
                         <bodyName>trunk</bodyName>
 			<topicName>ground_truth</topicName>

File: urdfs/flywheel.xacro (robot description, xacro)
@@ -2,4 +2,5 @@
 <robot xmlns:xacro="http://ros.org/wiki/xacro" name="solo">
 <!-- Things that are needed only for Gazebo (not the physical robot). These include sensor and controller plugin specifications -->
+<xacro:macro name="flywheel_train" params="radius">
     <xacro:include filename="$(find solo_description)/urdfs/flywheel.transmission.xacro"/>
     <xacro:include filename="$(find solo_description)/urdfs/flywheel.gazebo.xacro"/>
@@ -19,5 +20,5 @@
     <origin rpy="0 0 0" xyz="0 0 0.0"/>
     <geometry>
-    <cylinder length="0.05" radius="0.1"/>
+    <cylinder length="0.05" radius="${radius}"/>
     </geometry>
     </visual>
@@ -25,5 +26,5 @@
     <origin rpy="0 0 0" xyz="0 0 0.0"/>
     <geometry>
-     <cylinder length="0.05" radius="0.1"/>
+     <cylinder length="0.05" radius="${radius}"/>
     </geometry>
     </collision>    </link>
@@ -43,5 +44,5 @@
     <origin rpy="0 0 0" xyz="0 0 0.0"/>
     <geometry>
-    <cylinder length="0.05" radius="0.1"/>
+    <cylinder length="0.05" radius="${radius}"/>
     </geometry>
     </visual>
@@ -49,5 +50,5 @@
     <origin rpy="0 0 0" xyz="0 0 0.0"/>
     <geometry>
-     <cylinder length="0.05" radius="0.1"/>
+     <cylinder length="0.05" radius="${radius}"/>
     </geometry>
     </collision>
@@ -68,5 +69,5 @@
     <origin rpy="0 0 0" xyz="0 0 0.0"/>
     <geometry>
-    <cylinder length="0.05" radius="0.1"/>
+    <cylinder length="0.05" radius="${radius}"/>
     </geometry>
     </visual>
@@ -74,5 +75,5 @@
     <origin rpy="0 0 0" xyz="0 0 0"/>
     <geometry>
-     <cylinder length="0.05" radius="0.1"/>
+    <cylinder length="0.05" radius="${radius}"/>
     </geometry>
     </collision>
@@ -93,5 +94,5 @@
         <origin rpy="0 0 0" xyz="0 0 0.0"/>
         <geometry>
-        <cylinder length="0.05" radius="0.1"/>
+        <cylinder length="0.05" radius="${radius}"/>
         </geometry>
         </visual>
@@ -99,5 +100,5 @@
         <origin rpy="0 0 0" xyz="0 0 0.0"/>
         <geometry>
-         <cylinder length="0.05" radius="0.1"/>
+        <cylinder length="0.05" radius="${radius}"/>
         </geometry>
         </collision>
@@ -105,3 +106,4 @@
     <xacro:flywheel_transmission/>
     <xacro:flywheel_gazebo/>
+</xacro:macro>
 </robot>

File: urdfs/leg.gazebo.xacro (robot description, xacro)
@@ -8,5 +8,5 @@
                         <gazebo>
                                 <plugin name="${name}_haa_sensor" filename="libgazebo_ros_ft_sensor.so">
-                                        <robotNamespace>/solo12/internal_wrench/</robotNamespace>
+                                        <robotNamespace>/solo/internal_wrench/</robotNamespace>
                                         <updateRate>100.0</updateRate>
                                         <topicName>${name}_haa_joint</topicName>
@@ -21,5 +21,5 @@
                         <gazebo>
                                 <plugin name="${name}_kfe_sensor" filename="libgazebo_ros_ft_sensor.so">
-                                        <robotNamespace>/solo12/internal_wrench/</robotNamespace>
+                                        <robotNamespace>/solo/internal_wrench/</robotNamespace>
                                         <updateRate>100.0</updateRate>
                                         <topicName>${name}_kfe_joint</topicName>
@@ -34,5 +34,5 @@
                         <gazebo>
                                 <plugin name="${name}_hfe_sensor" filename="libgazebo_ros_ft_sensor.so">
-                                        <robotNamespace>/solo12/internal_wrench/</robotNamespace>
+                                        <robotNamespace>/solo/internal_wrench/</robotNamespace>
                                         <updateRate>100.0</updateRate>
                                         <topicName>${name}_hfe_joint</topicName>
@@ -66,5 +66,5 @@
                 because gazebo lumps the fake footframe with the real parent link, the normals are in the world frame-->
                  <plugin name="${name}_shin_bumper" filename="libgazebo_ros_bumper.so">
-                  <bumperTopicName>/solo12/${name}_shin_bumper</bumperTopicName>
+                  <bumperTopicName>/solo/${name}_shin_bumper</bumperTopicName>
                 </plugin>
             </sensor>
@@ -86,6 +86,6 @@
                                 because gazebo lumps the fake footframe with the real parent link, the normals are in the world frame-->
                                 <plugin name="${name}_foot_bumper" filename="libgazebo_ros_bumper.so">
-                                        <bumperTopicName>/solo12/${name}_foot_bumper</bumperTopicName>
-                                        <robotNamespace>solo12</robotNamespace>
+                                        <bumperTopicName>/solo/${name}_foot_bumper</bumperTopicName>
+                                        <robotNamespace>solo</robotNamespace>
                                 </plugin>
                         </sensor>

File: xacro/solo.srdf.xacro (robot description, xacro)
@@ -1,3 +1,3 @@
-<robot name="solo12" xmlns:xacro="http://ros.org/wiki/xacro">
+<robot name="solo" xmlns:xacro="http://ros.org/wiki/xacro">
   <group name="base">
     <link name="base_link"/>

File: xacro/solo.urdf.xacro (robot description, xacro)
@@ -1,8 +1,9 @@
 <?xml version="1.0" ?>
-<robot name="solo12"
+<robot name="solo"
   xmlns:controller="http://playerstage.sourceforge.net/gazebo/xmlschema/#controller"
   xmlns:interface="http://ros.org/wiki/xacro"
   xmlns:sensor="http://playerstage.sourceforge.net/gazebo/xmlschema/#sensor"
   xmlns:xacro="http://ros.org/wiki/xacro">
+  <xacro:arg name="fly" default="false"/>
   <xacro:arg name="load_force_sensors" default="false"/>
   <xacro:property name="color_name" value="grey" />
@@ -39,5 +40,5 @@
 				      <mesh filename="package://solo_description/meshes/stl/with_foot/solo_body.stl"/>
 				    </geometry>
-				    <material name="${color_name}">
+                                    <material name="${color_name}">
 				        <color rgba="${color} ${opacity}"/>
 				    </material>
@@ -60,6 +61,9 @@
  	 <!-- Include the legs -->
   	<xacro:include filename="$(find solo_description)/urdfs/leg.xacro"/>
-    <!-- Include flywheel -->
-    <xacro:include filename="$(find solo_description)/urdfs/flywheel.xacro"/>
+        <!-- Include flywheel -->
+        <xacro:if value="$(arg fly)">
+              <xacro:include filename="$(find solo_description)/urdfs/flywheel.xacro"/>
+                 <xacro:flywheel_train radius="0.05" />
+        </xacro:if>
   <!-- Include the front left leg -->
   <xacro:leg
