Commit message: removed load sensors and generalized the robot name for the libgazebo_ros_control

File: gazebo/gazebo.urdf.xacro (robot description, xacro)
@@ -1,5 +1,6 @@
 <?xml version="1.0"?>
 <robot xmlns:xacro="http://ros.org/wiki/xacro">
-<xacro:arg name="task_period" default="0.004"/>
+<xacro:arg name="task_period" default="0.004" />
+<xacro:arg name="robot_name" default="solo" />
 	<gazebo>
 		<plugin name="gazebo_ros_controller_manager" filename="libgazebo_ros_control.so">
@@ -11,5 +12,5 @@
 		</plugin>
 		<plugin filename="libgazebo_ros_p3d.so" name="gazebo_ros_p3d">
-                        <robotNamespace>/solo</robotNamespace>
+                        <robotNamespace>/$(arg robot_name)</robotNamespace>
                         <bodyName>trunk</bodyName>
 			<topicName>ground_truth</topicName>

File: robots/solo.urdf.xacro (robot description, xacro)
@@ -5,4 +5,5 @@
     <xacro:property name="opacity" value="1.0" />
     <xacro:arg name="flywheel" default="false"/>
+    <!--- new_gazebo_version should be false by default because pinocchio needs it!-->
     <xacro:arg name="flywheel2" default="true"/>
     <xacro:arg name="angle_deg" default="0.0"/>
@@ -11,4 +12,5 @@
     <xacro:include filename="$(find solo_description)/gazebo/gazebo.urdf.xacro">
         <xacro:arg name="task_period" value="$(arg task_period)"/>
+	<xacro:arg name="robot_name" value="$(arg robot_name)"/>
     </xacro:include>
     <!-- BASE LINK -->
@@ -84,6 +86,5 @@
     color_name="${color_name}"
     color="${color}"
-    opacity="${opacity}"
-    load_force_sensors="$(arg load_force_sensors)"/>
+    opacity="${opacity}"/>
     <!-- RIGHT FRONT LEG -->
     <xacro:leg
@@ -94,6 +95,5 @@
     color_name="${color_name}"
     color="${color}"
-    opacity="${opacity}"
-    load_force_sensors="$(arg load_force_sensors)"/>
+    opacity="${opacity}"/>
     <!-- LEFT HIND LEG -->
     <xacro:leg
@@ -104,6 +104,5 @@
     color_name="${color_name}"
     color="${color}"
-    opacity="${opacity}"
-    load_force_sensors="$(arg load_force_sensors)"/>
+    opacity="${opacity}"/>
     <!-- RIGHT HIND LEG -->
     <xacro:leg
@@ -114,5 +113,4 @@
     color_name="${color_name}"
     color="${color}"
-    opacity="${opacity}"
-    load_force_sensors="$(arg load_force_sensors)"/>
+    opacity="${opacity}"/>
 </robot>

File: urdfs/leg.gazebo.xacro (robot description, xacro)
@@ -1,44 +1,14 @@
 <?xml version="1.0"?>
 <robot xmlns:xacro="http://ros.org/wiki/xacro">
-        <xacro:macro name="leg_gazebo" params="name load_force_sensors">
+        <xacro:macro name="leg_gazebo" params="name">
                 <gazebo reference="${name}_haa_joint">
                         <provideFeedback>true</provideFeedback>
                 </gazebo>
-                <xacro:if value="${load_force_sensors}">
-                        <gazebo>
-                                <plugin name="${name}_haa_sensor" filename="libgazebo_ros_ft_sensor.so">
-                                        <robotNamespace>/solo/internal_wrench/</robotNamespace>
-                                        <updateRate>100.0</updateRate>
-                                        <topicName>${name}_haa_joint</topicName>
-                                        <jointName>${name}_haa_joint</jointName>
-                                </plugin>
-                        </gazebo>
-                </xacro:if>
                 <gazebo reference="${name}_kfe_joint">
                         <provideFeedback>true</provideFeedback>
                 </gazebo>
-                <xacro:if value="${load_force_sensors}">
-                        <gazebo>
-                                <plugin name="${name}_kfe_sensor" filename="libgazebo_ros_ft_sensor.so">
-                                        <robotNamespace>/solo/internal_wrench/</robotNamespace>
-                                        <updateRate>100.0</updateRate>
-                                        <topicName>${name}_kfe_joint</topicName>
-                                        <jointName>${name}_kfe_joint</jointName>
-                                </plugin>
-                        </gazebo>
-                </xacro:if>
                 <gazebo reference="${name}_hfe_joint">
                         <provideFeedback>true</provideFeedback>
                 </gazebo>
-                <xacro:if value="${load_force_sensors}">
-                        <gazebo>
-                                <plugin name="${name}_hfe_sensor" filename="libgazebo_ros_ft_sensor.so">
-                                        <robotNamespace>/solo/internal_wrench/</robotNamespace>
-                                        <updateRate>100.0</updateRate>
-                                        <topicName>${name}_hfe_joint</topicName>
-                                        <jointName>${name}_hfe_joint</jointName>
-                                </plugin>
-                        </gazebo>
-                </xacro:if>
                 <gazebo reference="${name}_upperleg">
                         <kp>1000000.0</kp>

File: urdfs/leg.xacro (robot description, xacro)
@@ -20,5 +20,5 @@
     <!-- This macro has for purpose to define a leg -->
     <xacro:macro name="leg" params="prefix is_front is_right has_side_motion
-                                  color_name color opacity load_force_sensors">
+                                  color_name color opacity">
         <!-- Solo12 -->
         <xacro:if value="${has_side_motion}">
@@ -456,5 +456,5 @@
         <!-- Extensions -->
         <xacro:leg_transmission name="${prefix}"/>
-        <xacro:leg_gazebo name="${prefix}" load_force_sensors="${load_force_sensors}"/>
+        <xacro:leg_gazebo name="${prefix}"/>
     </xacro:macro>
 </robot>

Commit message: fixing propagation of robot_name to bumpers and groundtruth

File: gazebo/gazebo.urdf.xacro (robot description, xacro)
@@ -6,5 +6,5 @@
 		<plugin name="gazebo_ros_controller_manager" filename="libgazebo_ros_control.so">
 			<!-- if task_period is smaller than sim max_step_size (in world file) it is clamped to that value!!!!!!-->
-			<robotNamespace>/solo</robotNamespace>
+			<robotNamespace>/$(arg robot_name)</robotNamespace>
 			<robotSimType>gazebo_ros_control/DefaultRobotHWSim</robotSimType>
 			<legacyModeNS>true</legacyModeNS>

File: robots/solo.urdf.xacro (robot description, xacro)
@@ -7,6 +7,6 @@
     <!--- new_gazebo_version should be false by default because pinocchio needs it!-->
     <xacro:arg name="flywheel2" default="false"/>
+    <xacro:arg name="robot_name" default="solo_fw"/>
     <xacro:arg name="angle_deg" default="0.0"/>
-    <xacro:arg name="load_force_sensors" default="false"/>
     <xacro:arg name="new_gazebo_version" default="false"/>
     <xacro:include filename="$(find solo_description)/gazebo/gazebo.urdf.xacro">
@@ -86,5 +86,6 @@
     color_name="${color_name}"
     color="${color}"
-    opacity="${opacity}"/>
+    opacity="${opacity}"
+    robot_name="$(arg robot_name)"/>
     <!-- RIGHT FRONT LEG -->
     <xacro:leg
@@ -95,5 +96,6 @@
     color_name="${color_name}"
     color="${color}"
-    opacity="${opacity}"/>
+    opacity="${opacity}"
+    robot_name="$(arg robot_name)"/>
     <!-- LEFT HIND LEG -->
     <xacro:leg
@@ -104,5 +106,6 @@
     color_name="${color_name}"
     color="${color}"
-    opacity="${opacity}"/>
+    opacity="${opacity}"
+    robot_name="$(arg robot_name)"/>
     <!-- RIGHT HIND LEG -->
     <xacro:leg
@@ -113,4 +116,5 @@
     color_name="${color_name}"
     color="${color}"
-    opacity="${opacity}"/>
+    opacity="${opacity}"
+    robot_name="$(arg robot_name)"/>
 </robot>

File: urdfs/leg.gazebo.xacro (robot description, xacro)
@@ -1,5 +1,5 @@
 <?xml version="1.0"?>
 <robot xmlns:xacro="http://ros.org/wiki/xacro">
-        <xacro:macro name="leg_gazebo" params="name">
+        <xacro:macro name="leg_gazebo" params="name robot_name">
                 <gazebo reference="${name}_haa_joint">
                         <provideFeedback>true</provideFeedback>
@@ -36,5 +36,5 @@
                 because gazebo lumps the fake footframe with the real parent link, the normals are in the world frame-->
                  <plugin name="${name}_shin_bumper" filename="libgazebo_ros_bumper.so">
-                  <bumperTopicName>/solo/${name}_shin_bumper</bumperTopicName>
+                  <bumperTopicName>/${robot_name}/${name}_shin_bumper</bumperTopicName>
                 </plugin>
             </sensor>
@@ -56,5 +56,5 @@
                                 because gazebo lumps the fake footframe with the real parent link, the normals are in the world frame-->
                                 <plugin name="${name}_foot_bumper" filename="libgazebo_ros_bumper.so">
-                                        <bumperTopicName>/solo/${name}_foot_bumper</bumperTopicName>
+                                        <bumperTopicName>/${robot_name}/${name}_foot_bumper</bumperTopicName>
                                         <!--robotNamespace>solo</robotNamespace-->
                                         <frameName>${name}_foot</frameName>

File: urdfs/leg.xacro (robot description, xacro)
@@ -20,5 +20,5 @@
     <!-- This macro has for purpose to define a leg -->
     <xacro:macro name="leg" params="prefix is_front is_right has_side_motion
-                                  color_name color opacity">
+                                  color_name color opacity robot_name">
         <!-- Solo12 -->
         <xacro:if value="${has_side_motion}">
@@ -456,5 +456,5 @@
         <!-- Extensions -->
         <xacro:leg_transmission name="${prefix}"/>
-        <xacro:leg_gazebo name="${prefix}"/>
+        <xacro:leg_gazebo name="${prefix}" robot_name="${robot_name}"/>
     </xacro:macro>
 </robot>
